Commit message: Audit all examples, fix geometry and training, publish MoveIt configs and GIFs

File: examples/04_scara/robot.urdf (robot description, URDF)
Before this commit: robot scara, 5 links, 4 joints
Links:
- link base_link: mass 1.017876 -> 1.781283; geometry collision cylinder length=0.35 radius=0.06; visual cylinder length=0.35 radius=0.06
Joints:
- joint joint_1: origin xyz=0 0 0.2 rpy=0 0 0 -> xyz=0 0 0.39 rpy=0 0 0

File: examples/05_diff_drive/robot.urdf (robot description, URDF)
Before this commit: robot diff_drive_robot, 4 links, 3 joints
Joints:
- joint left_wheel_joint: limit (none) -> effort=50 velocity=2
- joint right_wheel_joint: limit (none) -> effort=50 velocity=2

File: examples/06_four_wheel/robot.urdf (robot description, URDF)
Before this commit: robot four_wheel_robot, 5 links, 4 joints
Joints:
- joint front_left_wheel_joint: limit (none) -> effort=50 velocity=2
- joint front_right_wheel_joint: limit (none) -> effort=50 velocity=2
- joint rear_left_wheel_joint: limit (none) -> effort=50 velocity=2
- joint rear_right_wheel_joint: limit (none) -> effort=50 velocity=2

File: examples/07_mecanum/robot.urdf (robot description, URDF)
Before this commit: robot mecanum_robot, 5 links, 4 joints
Joints:
- joint front_left_wheel_joint: limit (none) -> effort=50 velocity=2
- joint front_right_wheel_joint: limit (none) -> effort=50 velocity=2
- joint rear_left_wheel_joint: limit (none) -> effort=50 velocity=2
- joint rear_right_wheel_joint: limit (none) -> effort=50 velocity=2

File: examples/08_humanoid/robot.urdf (robot description, URDF)
Before this commit: robot humanoid_robot, 28 links, 27 joints
Joints:
- joint left_gripper_base_joint: origin xyz=0 0 -0.06 rpy=0 0 0 -> xyz=0 0 -0.06 rpy=3.141593 0 0
- joint right_gripper_base_joint: origin xyz=0 0 -0.06 rpy=0 0 0 -> xyz=0 0 -0.06 rpy=3.141593 0 0

File: examples/11_spider_scout/robot.urdf (robot description, URDF)
Before this commit: robot hexapod, 20 links, 19 joints
Joints:
- joint front_left_tibia_joint: origin xyz=0.1 0 0 rpy=0 1.570796 0 -> xyz=0.1 0 0 rpy=0 0 0
- joint front_right_tibia_joint: origin xyz=0.1 0 0 rpy=0 1.570796 0 -> xyz=0.1 0 0 rpy=0 0 0
- joint mid_left_tibia_joint: origin xyz=0.1 0 0 rpy=0 1.570796 0 -> xyz=0.1 0 0 rpy=0 0 0
- joint mid_right_tibia_joint: origin xyz=0.1 0 0 rpy=0 1.570796 0 -> xyz=0.1 0 0 rpy=0 0 0
- joint rear_left_tibia_joint: origin xyz=0.1 0 0 rpy=0 1.570796 0 -> xyz=0.1 0 0 rpy=0 0 0
- joint rear_right_tibia_joint: origin xyz=0.1 0 0 rpy=0 1.570796 0 -> xyz=0.1 0 0 rpy=0 0 0

File: examples/12_mars_rover/robot.urdf (robot description, URDF)
Before this commit: robot rover_arm, 17 links, 16 joints
Joints:
- joint front_left_wheel_joint: limit (none) -> effort=50 velocity=2
- joint front_right_wheel_joint: limit (none) -> effort=50 velocity=2
- joint rear_left_wheel_joint: limit (none) -> effort=50 velocity=2
- joint rear_right_wheel_joint: limit (none) -> effort=50 velocity=2

File: examples/13_battle_mech/robot.urdf (robot description, URDF)
Before this commit: robot humanoid_robot, 30 links, 29 joints
Links:
- removed link camera_1_link
- removed link imu_1_link
- removed link left_gripper_base
- removed link left_left_finger
- removed link left_right_finger
- removed link right_gripper_base
- removed link right_left_finger
- removed link right_right_finger
- added link arc_reactor, mass 0.025977; collision cylinder length=0.015 radius=0.035; visual cylinder length=0.015 radius=0.035
- added link left_boot_thruster, mass 0.025447; collision cylinder length=0.02 radius=0.03; visual cylinder length=0.02 radius=0.03
- added link left_palm_repulsor, mass 0.025447; collision cylinder length=0.02 radius=0.03; visual cylinder length=0.02 radius=0.03
- added link right_boot_thruster, mass 0.025447; collision cylinder length=0.02 radius=0.03; visual cylinder length=0.02 radius=0.03
- added link right_palm_repulsor, mass 0.025447; collision cylinder length=0.02 radius=0.03; visual cylinder length=0.02 radius=0.03
- link left_forearm: geometry collision cylinder length=0.22 radius=0.04725; visual cylinder length=0.22 radius=0.04725
- link left_shin: geometry collision cylinder length=0.2 radius=0.054; visual cylinder length=0.2 radius=0.054
- link left_thigh: geometry collision cylinder length=0.2 radius=0.06075; visual cylinder length=0.2 radius=0.06075
- link left_upper_arm: geometry collision cylinder length=0.22 radius=0.04725; visual cylinder length=0.22 radius=0.04725
- link right_forearm: geometry collision cylinder length=0.22 radius=0.04725; visual cylinder length=0.22 radius=0.04725
- link right_shin: geometry collision cylinder length=0.2 radius=0.054; visual cylinder length=0.2 radius=0.054
- link right_thigh: geometry collision cylinder length=0.2 radius=0.06075; visual cylinder length=0.2 radius=0.06075
- link right_upper_arm: geometry collision cylinder length=0.22 radius=0.04725; visual cylinder length=0.22 radius=0.04725
Joints:
- removed joint camera_1_joint
- removed joint imu_1_joint
- removed joint left_gripper_base_joint
- removed joint left_left_finger_joint
- removed joint left_right_finger_joint
- removed joint right_gripper_base_joint
- removed joint right_left_finger_joint
- removed joint right_right_finger_joint
- added joint arc_reactor_joint: type fixed, parent torso, child arc_reactor, origin xyz=0.085 0 0.62 rpy=0 1.570796 0
- added joint left_boot_thruster_joint: type fixed, parent left_foot, child left_boot_thruster, origin xyz=-0.04 0 -0.03 rpy=0 0 0
- added joint left_palm_repulsor_joint: type fixed, parent left_wrist_3, child left_palm_repulsor, origin xyz=0 0 -0.07 rpy=0 0 0
- added joint right_boot_thruster_joint: type fixed, parent right_foot, child right_boot_thruster, origin xyz=-0.04 0 -0.03 rpy=0 0 0
- added joint right_palm_repulsor_joint: type fixed, parent right_wrist_3, child right_palm_repulsor, origin xyz=0 0 -0.07 rpy=0 0 0
- joint left_arm_joint_1: origin xyz=0 0.175 0.77 rpy=0 0 0 -> xyz=0 0.196 0.77 rpy=0 0 0
- joint right_arm_joint_1: origin xyz=0 -0.175 0.77 rpy=0 0 0 -> xyz=0 -0.196 0.77 rpy=0 0 0

File: examples/15_wall_e/robot.urdf (robot description, URDF)
Before this commit: robot wall_e, 23 links, 22 joints
Joints:
- joint left_front_wheel_joint: limit (none) -> effort=50 velocity=2
- joint left_rear_wheel_joint: limit (none) -> effort=50 velocity=2
- joint right_front_wheel_joint: limit (none) -> effort=50 velocity=2
- joint right_rear_wheel_joint: limit (none) -> effort=50 velocity=2

File: examples/16_eva/robot.urdf (robot description, URDF)
Before this commit: robot eva, 8 links, 7 joints
Links:
- link body: geometry collision cylinder length=0.3 radius=0.16; collision sphere radius=0.16
- link head: geometry collision cylinder length=0.1 radius=0.11; collision sphere radius=0.11
- link left_arm: geometry collision cylinder length=0.28 radius=0.06; collision sphere radius=0.06
- link right_arm: geometry collision cylinder length=0.28 radius=0.06; collision sphere radius=0.06

File: examples/17_baymax/robot.urdf (robot description, URDF)
Before this commit: robot baymax, 16 links, 15 joints
Links:
- link left_elbow: geometry collision cylinder length=0.005 radius=0.063; collision sphere radius=0.063
- link left_forearm: geometry collision cylinder length=0.094 radius=0.063; collision sphere radius=0.063
- link left_shin: geometry collision cylinder length=0.056 radius=0.072; collision sphere radius=0.072
- link left_shoulder: geometry collision cylinder length=0.005 radius=0.063; collision sphere radius=0.063
- link left_thigh: geometry collision cylinder length=0.038 radius=0.081; collision sphere radius=0.081
- link left_upper_arm: geometry collision cylinder length=0.094 radius=0.063; collision sphere radius=0.063
- link right_elbow: geometry collision cylinder length=0.005 radius=0.063; collision sphere radius=0.063
- link right_forearm: geometry collision cylinder length=0.094 radius=0.063; collision sphere radius=0.063
- link right_shin: geometry collision cylinder length=0.056 radius=0.072; collision sphere radius=0.072
- link right_shoulder: geometry collision cylinder length=0.005 radius=0.063; collision sphere radius=0.063
- link right_thigh: geometry collision cylinder length=0.038 radius=0.081; collision sphere radius=0.081
- link right_upper_arm: geometry collision cylinder length=0.094 radius=0.063; collision sphere radius=0.063
- link torso: geometry collision cylinder length=0.162 radius=0.154; collision sphere radius=0.154
Joints:
- joint left_arm_joint_1: origin xyz=0 0.175 0.77 rpy=0 0 0 -> xyz=0 0.27 0.77 rpy=0 0 0
- joint right_arm_joint_1: origin xyz=0 -0.175 0.77 rpy=0 0 0 -> xyz=0 -0.27 0.77 rpy=0 0 0
