Commit message: Replace dragging differential-drive supports with passive swivel casters

File: examples/05_diff_drive/robot.urdf (robot description, URDF)
Before this commit: robot diff_drive_robot, 14 links, 13 joints
Links:
- removed link caster
- removed link rear_caster
- added link front_caster_fork, mass 0.03; collision cylinder length=0.04 radius=0.008; visual cylinder length=0.04 radius=0.008
- added link front_caster_wheel, mass 0.08; collision cylinder length=0.018 radius=0.03; visual cylinder length=0.018 radius=0.03
- added link rear_caster_fork, mass 0.03; collision cylinder length=0.04 radius=0.008; visual cylinder length=0.04 radius=0.008
- added link rear_caster_wheel, mass 0.08; collision cylinder length=0.018 radius=0.03; visual cylinder length=0.018 radius=0.03
Joints:
- removed joint caster_joint
- removed joint rear_caster_mount
- added joint front_caster_bearing: type continuous, parent front_caster_fork, child front_caster_wheel, origin xyz=-0.018 0 -0.05 rpy=0 0 0, axis 0 1 0, limit effort=0.01 velocity=100
- added joint front_caster_swivel: type continuous, parent base_link, child front_caster_fork, origin xyz=0.15 0 0.08 rpy=0 0 0, axis 0 0 1, limit effort=0.01 velocity=100
- added joint rear_caster_bearing: type continuous, parent rear_caster_fork, child rear_caster_wheel, origin xyz=-0.018 0 -0.05 rpy=0 0 0, axis 0 1 0, limit effort=0.01 velocity=100
- added joint rear_caster_swivel: type continuous, parent base_link, child rear_caster_fork, origin xyz=-0.15 0 0.08 rpy=0 0 0, axis 0 0 1, limit effort=0.01 velocity=100

Commit message: Local free web generation and researched robot mechanism improvements (#8)
* Make generation local and improve researched robot mechanisms and validation

* Replace dragging differential-drive supports with passive swivel casters

---------

Co-authored-by: megazron <megazron@users.noreply.github.com>

File: examples/05_diff_drive/robot.urdf (robot description, URDF)
Before this commit: robot diff_drive_robot, 4 links, 3 joints
Links:
- removed link caster
- added link base_link_front_panel, mass 0.27702; collision box size=0.003 0.3 0.114; visual box size=0.003 0.3 0.114
- added link base_link_left_panel, mass 0.36382; collision box size=0.394 0.003 0.114; visual box size=0.394 0.003 0.114
- added link base_link_rear_panel, mass 0.27702; collision box size=0.003 0.3 0.114; visual box size=0.003 0.3 0.114
- added link base_link_right_panel, mass 0.36382; collision box size=0.394 0.003 0.114; visual box size=0.394 0.003 0.114
- added link base_link_service_lid, mass 0.945789; collision box size=0.4 0.3 0.003; visual mesh filename=package://diff_drive_robot/meshes/base_link_service_lid.stl
- added link base_link_standoff_fl, mass 0.02; collision box size=0.008 0.008 0.114; visual mesh filename=package://diff_drive_robot/meshes/base_link_standoff_fl.stl
- added link base_link_standoff_fr, mass 0.02; collision box size=0.008 0.008 0.114; visual mesh filename=package://diff_drive_robot/meshes/base_link_standoff_fr.stl
- added link base_link_standoff_rl, mass 0.02; collision box size=0.008 0.008 0.114; visual mesh filename=package://diff_drive_robot/meshes/base_link_standoff_rl.stl
- added link base_link_standoff_rr, mass 0.02; collision box size=0.008 0.008 0.114; visual mesh filename=package://diff_drive_robot/meshes/base_link_standoff_rr.stl
- added link front_caster_fork, mass 0.03; collision cylinder length=0.04 radius=0.008; visual cylinder length=0.04 radius=0.008
- added link front_caster_wheel, mass 0.08; collision cylinder length=0.018 radius=0.03; visual cylinder length=0.018 radius=0.03
- added link rear_caster_fork, mass 0.03; collision cylinder length=0.04 radius=0.008; visual cylinder length=0.04 radius=0.008
- added link rear_caster_wheel, mass 0.08; collision cylinder length=0.018 radius=0.03; visual cylinder length=0.018 radius=0.03
- link base_link: mass 6.48 -> 0.971709; geometry collision box size=0.4 0.3 0.003; visual mesh filename=package://diff_drive_robot/meshes/base_link.stl
Joints:
- removed joint caster_joint
- added joint base_link_front_panel_mount: type fixed, parent base_link, child base_link_front_panel, origin xyz=0 0 0 rpy=0 0 0
- added joint base_link_left_panel_mount: type fixed, parent base_link, child base_link_left_panel, origin xyz=0 0 0 rpy=0 0 0
- added joint base_link_rear_panel_mount: type fixed, parent base_link, child base_link_rear_panel, origin xyz=0 0 0 rpy=0 0 0
- added joint base_link_right_panel_mount: type fixed, parent base_link, child base_link_right_panel, origin xyz=0 0 0 rpy=0 0 0
- added joint base_link_service_lid_mount: type fixed, parent base_link, child base_link_service_lid, origin xyz=0 0 0 rpy=0 0 0
- added joint base_link_standoff_fl_mount: type fixed, parent base_link, child base_link_standoff_fl, origin xyz=0 0 0 rpy=0 0 0
- added joint base_link_standoff_fr_mount: type fixed, parent base_link, child base_link_standoff_fr, origin xyz=0 0 0 rpy=0 0 0
- added joint base_link_standoff_rl_mount: type fixed, parent base_link, child base_link_standoff_rl, origin xyz=0 0 0 rpy=0 0 0
- added joint base_link_standoff_rr_mount: type fixed, parent base_link, child base_link_standoff_rr, origin xyz=0 0 0 rpy=0 0 0
- added joint front_caster_bearing: type continuous, parent front_caster_fork, child front_caster_wheel, origin xyz=-0.018 0 -0.05 rpy=0 0 0, axis 0 1 0, limit effort=0.01 velocity=100
- added joint front_caster_swivel: type continuous, parent base_link, child front_caster_fork, origin xyz=0.15 0 0.08 rpy=0 0 0, axis 0 0 1, limit effort=0.01 velocity=100
- added joint rear_caster_bearing: type continuous, parent rear_caster_fork, child rear_caster_wheel, origin xyz=-0.018 0 -0.05 rpy=0 0 0, axis 0 1 0, limit effort=0.01 velocity=100
- added joint rear_caster_swivel: type continuous, parent base_link, child rear_caster_fork, origin xyz=-0.15 0 0.08 rpy=0 0 0, axis 0 0 1, limit effort=0.01 velocity=100
- joint left_wheel_joint: limit effort=50 velocity=2 -> effort=2.5 velocity=12
- joint right_wheel_joint: limit effort=50 velocity=2 -> effort=2.5 velocity=12
