Commit message: feat: buildable BOM, CAD parts, training suite, sci-fi robots, viewer screenshots
Toward the goal of "describe a robot, download it, and start training it" as a
free, self-hostable service.

- components: real-world Bill of Materials sized to a cost budget (actuators by
  downstream torque, sensors, compute, power, structure); fits the budget across
  hobby/prosumer/research tiers
- cad: parametric OpenSCAD parts per link + assembly (mesh to STL)
- training-export: PyBullet + Gymnasium suite -- RL (PPO/SAC), imitation learning
  (demo collection + behaviour cloning), evaluation; task per robot class
- templates: hexapod (18 DOF) and rover+arm (mobile manipulator); NL routing for
  sci-fi prompts + inline sensor detection (LiDAR/camera/IMU) + budget parsing
- realistic link mass via effective printed density (was solid aluminium)
- web: Build/BOM tab with budget input, CAD/BOM/Train downloads, robust camera framing
- api + cli: /bom, /cad, /training endpoints; CLI writes BOM.md + cad/ + training/
- README: real viewer screenshots, sci-fi examples, buildability/CAD/training docs,
  free self-hostable positioning; 43 tests, 13 examples

File: examples/01_arm_2dof/robot.urdf (robot description, URDF)
Before this commit: robot arm_2dof, 6 links, 5 joints
Links:
- link base_link: mass 3.664354 -> 0.610726
- link gripper_base: mass 0.3888 -> 0.0648
- link left_finger: mass 0.0486 -> 0.02
- link right_finger: mass 0.0486 -> 0.02
- link shoulder: mass 1.357168 -> 0.226195
- link upper_arm: mass 3.39292 -> 0.565487

File: examples/02_arm_6dof/robot.urdf (robot description, URDF)
Before this commit: robot arm_6dof, 10 links, 9 joints
Links:
- link base_link: mass 3.664354 -> 0.610726
- link forearm: mass 3.39292 -> 0.565487
- link gripper_base: mass 0.3888 -> 0.0648
- link left_finger: mass 0.0486 -> 0.02
- link right_finger: mass 0.0486 -> 0.02
- link shoulder: mass 1.357168 -> 0.226195
- link upper_arm: mass 3.39292 -> 0.565487
- link wrist_1: mass 0.760014 -> 0.126669
- link wrist_2: mass 0.922874 -> 0.153812
- link wrist_3: mass 1.085734 -> 0.180956

File: examples/03_arm_7dof/robot.urdf (robot description, URDF)
Before this commit: robot arm_7dof, 11 links, 10 joints
Links:
- link base_link: mass 3.664354 -> 0.610726
- link forearm: mass 3.39292 -> 0.565487
- link gripper_base: mass 0.3888 -> 0.0648
- link left_finger: mass 0.0486 -> 0.02
- link link_4: mass 1.221451 -> 0.203575
- link right_finger: mass 0.0486 -> 0.02
- link shoulder: mass 1.357168 -> 0.226195
- link upper_arm: mass 3.39292 -> 0.565487
- link wrist_1: mass 0.760014 -> 0.126669
- link wrist_2: mass 0.922874 -> 0.153812
- link wrist_3: mass 1.085734 -> 0.180956

File: examples/04_scara/robot.urdf (robot description, URDF)
Before this commit: robot scara, 5 links, 4 joints
Links:
- link base_link: mass 6.107256 -> 1.017876
- link forearm: mass 1.526814 -> 0.254469
- link spindle: mass 0.40715 -> 0.067858
- link tool: mass 0.057256 -> 0.02
- link upper_arm: mass 2.597704 -> 0.432951

File: examples/05_diff_drive/robot.urdf (robot description, URDF)
Before this commit: robot diff_drive_robot, 4 links, 3 joints
Links:
- link base_link: mass 38.88 -> 6.48
- link caster: mass 0.527667 -> 0.087944
- link left_wheel: mass 1.221451 -> 0.203575
- link right_wheel: mass 1.221451 -> 0.203575

File: examples/06_four_wheel/robot.urdf (robot description, URDF)
Before this commit: robot four_wheel_robot, 5 links, 4 joints
Links:
- link base_link: mass 38.88 -> 6.48
- link front_left_wheel: mass 1.221451 -> 0.203575
- link front_right_wheel: mass 1.221451 -> 0.203575
- link rear_left_wheel: mass 1.221451 -> 0.203575
- link rear_right_wheel: mass 1.221451 -> 0.203575

File: examples/07_mecanum/robot.urdf (robot description, URDF)
Before this commit: robot mecanum_robot, 5 links, 4 joints
Links:
- link base_link: mass 38.88 -> 6.48
- link front_left_wheel: mass 1.221451 -> 0.203575
- link front_right_wheel: mass 1.221451 -> 0.203575
- link rear_left_wheel: mass 1.221451 -> 0.203575
- link rear_right_wheel: mass 1.221451 -> 0.203575

File: examples/08_humanoid/robot.urdf (robot description, URDF)
Before this commit: robot humanoid_robot, 22 links, 21 joints
Links:
- link head: mass 8.244796 -> 1.374133
- link left_elbow: mass 0.623449 -> 0.103908
- link left_forearm: mass 2.28598 -> 0.380997
- link left_gripper_base: mass 0.3888 -> 0.0648
- link left_left_finger: mass 0.0486 -> 0.02
- link left_right_finger: mass 0.0486 -> 0.02
- link left_shoulder: mass 0.623449 -> 0.103908
- link left_upper_arm: mass 2.28598 -> 0.380997
- link left_wrist_1: mass 0.623449 -> 0.103908
- link left_wrist_2: mass 0.623449 -> 0.103908
- link left_wrist_3: mass 0.623449 -> 0.103908
- link right_elbow: mass 0.623449 -> 0.103908
- link right_forearm: mass 2.28598 -> 0.380997
- link right_gripper_base: mass 0.3888 -> 0.0648
- link right_left_finger: mass 0.0486 -> 0.02
- link right_right_finger: mass 0.0486 -> 0.02
- link right_shoulder: mass 0.623449 -> 0.103908
- link right_upper_arm: mass 2.28598 -> 0.380997
- link right_wrist_1: mass 0.623449 -> 0.103908
- link right_wrist_2: mass 0.623449 -> 0.103908
- link right_wrist_3: mass 0.623449 -> 0.103908
- link torso: mass 43.5456 -> 7.2576

File: examples/09_gripper/robot.urdf (robot description, URDF)
Before this commit: robot parallel_gripper, 4 links, 3 joints
Links:
- link base_link: mass 3.664354 -> 0.610726
- link gripper_base: mass 0.3888 -> 0.0648
- link left_finger: mass 0.0486 -> 0.02
- link right_finger: mass 0.0486 -> 0.02

File: examples/10_quadruped/robot.urdf (robot description, URDF)
Before this commit: robot quadruped, 13 links, 12 joints
Links:
- link base_link: mass 21.6 -> 3.6
- link front_left_hip: mass 0.381704 -> 0.063617
- link front_left_shin: mass 0.439722 -> 0.073287
- link front_left_thigh: mass 0.656869 -> 0.109478
- link front_right_hip: mass 0.381704 -> 0.063617
- link front_right_shin: mass 0.439722 -> 0.073287
- link front_right_thigh: mass 0.656869 -> 0.109478
- link rear_left_hip: mass 0.381704 -> 0.063617
- link rear_left_shin: mass 0.439722 -> 0.073287
- link rear_left_thigh: mass 0.656869 -> 0.109478
- link rear_right_hip: mass 0.381704 -> 0.063617
- link rear_right_shin: mass 0.439722 -> 0.073287
- link rear_right_thigh: mass 0.656869 -> 0.109478

Commit message: Verify rendered geometry and improve arm solids, control and MoveIt motion

File: examples/01_arm_2dof/robot.urdf (robot description, URDF)
Before this commit: robot arm_2dof, 20 links, 19 joints
Links:
- removed link shoulder_mount
- added link shoulder_mount_left, mass 0.02; collision box size=0.02 0.008 0.044; visual box size=0.02 0.008 0.044
- added link shoulder_mount_right, mass 0.02; collision box size=0.02 0.008 0.044; visual box size=0.02 0.008 0.044
- link shoulder: mass 0.199341 -> 0.21879; geometry collision cylinder length=0.182 radius=0.0288; collision cylinder length=0.25 radius=0.01152
- link upper_arm: mass 0.199341 -> 0.21879; geometry collision cylinder length=0.182 radius=0.0288; collision cylinder length=0.25 radius=0.01152
Joints:
- removed joint shoulder_mount_fixed
- added joint shoulder_mount_left_fixed: type fixed, parent base_link, child shoulder_mount_left, origin xyz=0 0 0 rpy=0 0 0
- added joint shoulder_mount_right_fixed: type fixed, parent base_link, child shoulder_mount_right, origin xyz=0 0 0 rpy=0 0 0

File: examples/02_arm_6dof/robot.urdf (robot description, URDF)
Before this commit: robot arm_6dof, 28 links, 27 joints
Links:
- link forearm: mass 0.199341 -> 0.21879; geometry collision cylinder length=0.182 radius=0.0288; collision cylinder length=0.25 radius=0.01152
- link shoulder: mass 0.032572 -> 0.043782; geometry collision cylinder length=0.052 radius=0.024; collision cylinder length=0.1 radius=0.0096
- link upper_arm: mass 0.199341 -> 0.21879; geometry collision cylinder length=0.182 radius=0.0288; collision cylinder length=0.25 radius=0.01152
- link wrist_1: geometry collision cylinder length=0.03248 radius=0.01344; collision cylinder length=0.056 radius=0.005376
- link wrist_2: geometry collision cylinder length=0.0392 radius=0.01632; collision cylinder length=0.068 radius=0.006528
- link wrist_3: mass 0.02 -> 0.022865; geometry collision cylinder length=0.044 radius=0.0192; collision cylinder length=0.08 radius=0.00768

File: examples/03_arm_7dof/robot.urdf (robot description, URDF)
Before this commit: robot arm_7dof, 30 links, 29 joints
Links:
- link forearm: mass 0.199341 -> 0.21879; geometry collision cylinder length=0.182 radius=0.0288; collision cylinder length=0.25 radius=0.01152
- link link_4: mass 0.023745 -> 0.032201; geometry collision cylinder length=0.048 radius=0.0216; collision cylinder length=0.09 radius=0.00864
- link shoulder: mass 0.032572 -> 0.043782; geometry collision cylinder length=0.052 radius=0.024; collision cylinder length=0.1 radius=0.0096
- link upper_arm: mass 0.199341 -> 0.21879; geometry collision cylinder length=0.182 radius=0.0288; collision cylinder length=0.25 radius=0.01152
- link wrist_1: geometry collision cylinder length=0.03248 radius=0.01344; collision cylinder length=0.056 radius=0.005376
- link wrist_2: geometry collision cylinder length=0.0392 radius=0.01632; collision cylinder length=0.068 radius=0.006528
- link wrist_3: mass 0.02 -> 0.022865; geometry collision cylinder length=0.044 radius=0.0192; collision cylinder length=0.08 radius=0.00768

File: examples/08_humanoid/robot.urdf (robot description, URDF)
Before this commit: robot humanoid_robot, 47 links, 46 joints
Links:
- link left_shin: mass 0.452389 -> 0.445604; geometry collision cylinder length=0.197 radius=0.04; visual cylinder length=0.197 radius=0.04
- link left_thigh: mass 0.572555 -> 0.563967; geometry collision cylinder length=0.197 radius=0.045; visual cylinder length=0.197 radius=0.045
- link right_shin: mass 0.452389 -> 0.445604; geometry collision cylinder length=0.197 radius=0.04; visual cylinder length=0.197 radius=0.04
- link right_thigh: mass 0.572555 -> 0.563967; geometry collision cylinder length=0.197 radius=0.045; visual cylinder length=0.197 radius=0.045
Joints:
- joint left_arm_joint_1: origin xyz=0 0.175 0.77 rpy=0 0 0 -> xyz=0 0.178 0.77 rpy=0 0 0
- joint right_arm_joint_1: origin xyz=0 -0.175 0.77 rpy=0 0 0 -> xyz=0 -0.178 0.77 rpy=0 0 0

File: examples/12_mars_rover/robot.urdf (robot description, URDF)
Before this commit: robot rover_arm, 44 links, 43 joints
Links:
- link forearm: mass 0.199341 -> 0.21879; geometry collision cylinder length=0.182 radius=0.0288; collision cylinder length=0.25 radius=0.01152
- link shoulder: mass 0.032572 -> 0.043782; geometry collision cylinder length=0.052 radius=0.024; collision cylinder length=0.1 radius=0.0096
- link upper_arm: mass 0.199341 -> 0.21879; geometry collision cylinder length=0.182 radius=0.0288; collision cylinder length=0.25 radius=0.01152
- link wrist_1: geometry collision cylinder length=0.03248 radius=0.01344; collision cylinder length=0.056 radius=0.005376
- link wrist_2: geometry collision cylinder length=0.0392 radius=0.01632; collision cylinder length=0.068 radius=0.006528
- link wrist_3: mass 0.02 -> 0.022865; geometry collision cylinder length=0.044 radius=0.0192; collision cylinder length=0.08 radius=0.00768

File: examples/13_battle_mech/robot.urdf (robot description, URDF)
Before this commit: robot battle_mech, 42 links, 41 joints
Links:
- link left_shin: mass 0.452389 -> 0.445604; geometry collision cylinder length=0.197 radius=0.054; visual cylinder length=0.197 radius=0.054
- link left_thigh: mass 0.572555 -> 0.563967; geometry collision cylinder length=0.197 radius=0.06075; visual cylinder length=0.197 radius=0.06075
- link right_shin: mass 0.452389 -> 0.445604; geometry collision cylinder length=0.197 radius=0.054; visual cylinder length=0.197 radius=0.054
- link right_thigh: mass 0.572555 -> 0.563967; geometry collision cylinder length=0.197 radius=0.06075; visual cylinder length=0.197 radius=0.06075
Joints:
- joint left_arm_joint_1: origin xyz=0 0.196 0.77 rpy=0 0 0 -> xyz=0 0.19936 0.77 rpy=0 0 0
- joint right_arm_joint_1: origin xyz=0 -0.196 0.77 rpy=0 0 0 -> xyz=0 -0.19936 0.77 rpy=0 0 0

File: examples/17_baymax/robot.urdf (robot description, URDF)
Before this commit: robot baymax, 22 links, 21 joints
Links:
- link left_shin: mass 1.130973 -> 1.114009; geometry collision cylinder length=0.053 radius=0.072; collision sphere radius=0.072
- link left_thigh: mass 1.431388 -> 1.409917; geometry collision cylinder length=0.035 radius=0.081; collision sphere radius=0.081
- link right_shin: mass 1.130973 -> 1.114009; geometry collision cylinder length=0.053 radius=0.072; collision sphere radius=0.072
- link right_thigh: mass 1.431388 -> 1.409917; geometry collision cylinder length=0.035 radius=0.081; collision sphere radius=0.081
