Commit message: Mark 43 refinement pass + MuJoCo gallery for every example
- Mark 43: sculpted pectoral loft, gold forearm/thigh/shin stripes, neck ring,
  larger pauldrons/knee/elbow caps, longer limb shells, gunmetal exo frame
- wearer mannequin: dark undersuit, head height corrected to the person's
  stature so the helmet closes around it
- docs/img/examples: ttr-mujoco render of all 17 examples, README gallery
- battery reports, MJCFs, renders and viewer screenshot regenerated

File: examples/14_iron_man_mark_43/robot.sim.urdf (robot description, URDF)
Before this commit: robot iron_man_mark_43, 125 links, 124 joints
Links:
- added link left_gauntlet_stripe, mass 0.03; collision box size=0.004853 0.032695 0.102794; visual mesh filename=meshes/left_gauntlet_stripe.stl
- added link left_shin_stripe, mass 0.05; collision box size=0.005233 0.042669 0.162674; visual mesh filename=meshes/left_shin_stripe.stl
- added link left_thigh_stripe, mass 0.05; collision box size=0.004525 0.037827 0.182634; visual mesh filename=meshes/left_thigh_stripe.stl
- added link neck_ring, mass 0.3; collision box size=0.16 0.16 0.025; visual mesh filename=meshes/neck_ring.stl
- added link right_gauntlet_stripe, mass 0.03; collision box size=0.004853 0.032695 0.102794; visual mesh filename=meshes/right_gauntlet_stripe.stl
- added link right_shin_stripe, mass 0.05; collision box size=0.005233 0.042669 0.162674; visual mesh filename=meshes/right_shin_stripe.stl
- added link right_thigh_stripe, mass 0.05; collision box size=0.004525 0.037827 0.182634; visual mesh filename=meshes/right_thigh_stripe.stl
- link left_bicep_clamshell: geometry collision box size=0.119616 0.039871 0.228308; visual mesh filename=meshes/left_bicep_clamshell.stl
- link left_bicep_sleeve: geometry collision box size=0.15959 0.15171 0.228306; visual mesh filename=meshes/left_bicep_sleeve.stl
- link left_calf_clamshell: geometry collision box size=0.154507 0.055798 0.327702; visual mesh filename=meshes/left_calf_clamshell.stl
- link left_chest_door: geometry collision box size=0.134852 0.240172 0.34; visual mesh filename=meshes/left_chest_door.stl
- link left_elbow_cap: geometry collision box size=0.117867 0.117867 0.043982; visual mesh filename=meshes/left_elbow_cap.stl
- link left_gauntlet_clamshell: geometry collision box size=0.105395 0.037654 0.189534; visual mesh filename=meshes/left_gauntlet_clamshell.stl
- link left_gauntlet_sleeve: geometry collision box size=0.14163 0.134065 0.189532; visual mesh filename=meshes/left_gauntlet_sleeve.stl
- link left_knee_cap: geometry collision box size=0.149828 0.149828 0.054978; visual mesh filename=meshes/left_knee_cap.stl
- link left_pauldron: geometry collision box size=0.269818 0.269818 0.094979; visual mesh filename=meshes/left_pauldron.stl
- link left_pauldron_edge: geometry collision box size=0.012145 0.091966 0.033932; visual mesh filename=meshes/left_pauldron_edge.stl
- link left_shin_shell: geometry collision box size=0.207453 0.196274 0.3277; visual mesh filename=meshes/left_shin_shell.stl
- link left_thigh_clamshell: geometry collision box size=0.180452 0.062313 0.343583; visual mesh filename=meshes/left_thigh_clamshell.stl
- link left_thigh_shell: geometry collision box size=0.241367 0.228928 0.343581; visual mesh filename=meshes/left_thigh_shell.stl
- link right_bicep_clamshell: geometry collision box size=0.119616 0.039871 0.228308; visual mesh filename=meshes/right_bicep_clamshell.stl
- link right_bicep_sleeve: geometry collision box size=0.15959 0.15171 0.228306; visual mesh filename=meshes/right_bicep_sleeve.stl
- link right_calf_clamshell: geometry collision box size=0.154506 0.055798 0.327702; visual mesh filename=meshes/right_calf_clamshell.stl
- link right_chest_door: geometry collision box size=0.134865 0.240172 0.34; visual mesh filename=meshes/right_chest_door.stl
- link right_elbow_cap: geometry collision box size=0.117867 0.117867 0.043982; visual mesh filename=meshes/right_elbow_cap.stl
- link right_gauntlet_clamshell: geometry collision box size=0.105394 0.037654 0.189534; visual mesh filename=meshes/right_gauntlet_clamshell.stl
- link right_gauntlet_sleeve: geometry collision box size=0.14163 0.134065 0.189532; visual mesh filename=meshes/right_gauntlet_sleeve.stl
- link right_knee_cap: geometry collision box size=0.149828 0.149828 0.054978; visual mesh filename=meshes/right_knee_cap.stl
- link right_pauldron: geometry collision box size=0.269818 0.269818 0.094979; visual mesh filename=meshes/right_pauldron.stl
- link right_pauldron_edge: geometry collision box size=0.012145 0.091966 0.033932; visual mesh filename=meshes/right_pauldron_edge.stl
- link right_shin_shell: geometry collision box size=0.207454 0.196274 0.3277; visual mesh filename=meshes/right_shin_shell.stl
- link right_thigh_clamshell: geometry collision box size=0.180452 0.062313 0.343583; visual mesh filename=meshes/right_thigh_clamshell.stl
- link right_thigh_shell: geometry collision box size=0.241367 0.228928 0.343581; visual mesh filename=meshes/right_thigh_shell.stl
Joints:
- added joint left_gauntlet_stripe_mount: type fixed, parent left_gauntlet_sleeve, child left_gauntlet_stripe, origin xyz=0.067 0 -0.09 rpy=0 0 0
- added joint left_shin_stripe_mount: type fixed, parent left_shin_shell, child left_shin_stripe, origin xyz=0.099 0 -0.16 rpy=0 0 0
- added joint left_thigh_stripe_mount: type fixed, parent left_thigh_shell, child left_thigh_stripe, origin xyz=0 0.116 -0.17 rpy=0 0 1.570796
- added joint neck_ring_mount: type fixed, parent spine_frame, child neck_ring, origin xyz=0.02 0 0.524 rpy=0 0 0
- added joint right_gauntlet_stripe_mount: type fixed, parent right_gauntlet_sleeve, child right_gauntlet_stripe, origin xyz=0.067 0 -0.09 rpy=0 0 0
- added joint right_shin_stripe_mount: type fixed, parent right_shin_shell, child right_shin_stripe, origin xyz=0.099 0 -0.16 rpy=0 0 0
- added joint right_thigh_stripe_mount: type fixed, parent right_thigh_shell, child right_thigh_stripe, origin xyz=0 -0.116 -0.17 rpy=0 0 -1.570796
- joint left_bicep_clamshell_hinge: origin xyz=0.037318 -0.115057 -0.04557 rpy=0 0 0 -> xyz=0.037318 -0.115057 -0.03906 rpy=0 0 0
- joint left_bicep_sleeve_mount: origin xyz=0 -0.05 -0.04557 rpy=0 0 0 -> xyz=0 -0.05 -0.03906 rpy=0 0 0
- joint left_calf_clamshell_hinge: origin xyz=0.048762 -0.130007 -0.05166 rpy=0 0 0 -> xyz=0.048762 -0.130007 -0.04305 rpy=0 0 0
- joint left_gauntlet_clamshell_hinge: origin xyz=0.03284 -0.10225 -0.033215 rpy=0 0 0 -> xyz=0.03284 -0.10225 -0.028105 rpy=0 0 0
- joint left_gauntlet_sleeve_mount: origin xyz=0 -0.045 -0.033215 rpy=0 0 0 -> xyz=0 -0.045 -0.028105 rpy=0 0 0
- joint left_pauldron_edge_mount: origin xyz=0.117 0 0.022 rpy=0 0 0 -> xyz=0.127 0 0.024 rpy=0 0 0
- joint left_pauldron_hinge: origin xyz=0 -0.02 0.025 rpy=-0.45 0 0 -> xyz=0 -0.02 0.02 rpy=-0.45 0 0
- joint left_shin_shell_mount: origin xyz=0 -0.045 -0.05166 rpy=0 0 0 -> xyz=0 -0.045 -0.04305 rpy=0 0 0
- joint left_thigh_clamshell_hinge: origin xyz=0.057221 -0.144754 -0.05145 rpy=0 0 0 -> xyz=0.057221 -0.144754 -0.042875 rpy=0 0 0
- joint left_thigh_shell_mount: origin xyz=0 -0.045 -0.05145 rpy=0 0 0 -> xyz=0 -0.045 -0.042875 rpy=0 0 0
- joint right_bicep_clamshell_hinge: origin xyz=0.037318 0.115057 -0.04557 rpy=0 0 0 -> xyz=0.037318 0.115057 -0.03906 rpy=0 0 0
- joint right_bicep_sleeve_mount: origin xyz=0 0.05 -0.04557 rpy=0 0 0 -> xyz=0 0.05 -0.03906 rpy=0 0 0
- joint right_calf_clamshell_hinge: origin xyz=0.048762 0.130007 -0.05166 rpy=0 0 0 -> xyz=0.048762 0.130007 -0.04305 rpy=0 0 0
- joint right_gauntlet_clamshell_hinge: origin xyz=0.03284 0.10225 -0.033215 rpy=0 0 0 -> xyz=0.03284 0.10225 -0.028105 rpy=0 0 0
- joint right_gauntlet_sleeve_mount: origin xyz=0 0.045 -0.033215 rpy=0 0 0 -> xyz=0 0.045 -0.028105 rpy=0 0 0
- joint right_pauldron_edge_mount: origin xyz=0.117 0 0.022 rpy=0 0 0 -> xyz=0.127 0 0.024 rpy=0 0 0
- joint right_pauldron_hinge: origin xyz=0 0.02 0.025 rpy=0.45 0 0 -> xyz=0 0.02 0.02 rpy=0.45 0 0
- joint right_shin_shell_mount: origin xyz=0 0.045 -0.05166 rpy=0 0 0 -> xyz=0 0.045 -0.04305 rpy=0 0 0
- joint right_thigh_clamshell_hinge: origin xyz=0.057221 0.144754 -0.05145 rpy=0 0 0 -> xyz=0.057221 0.144754 -0.042875 rpy=0 0 0
- joint right_thigh_shell_mount: origin xyz=0 0.045 -0.05145 rpy=0 0 0 -> xyz=0 0.045 -0.042875 rpy=0 0 0

File: examples/14_iron_man_mark_43/robot.urdf (robot description, URDF)
Before this commit: robot iron_man_mark_43, 125 links, 124 joints
Links:
- added link left_gauntlet_stripe, mass 0.03; collision box size=0.004853 0.032695 0.102794; visual mesh filename=package://iron_man_mark_43/meshes/left_gauntlet_stripe.stl
- added link left_shin_stripe, mass 0.05; collision box size=0.005233 0.042669 0.162674; visual mesh filename=package://iron_man_mark_43/meshes/left_shin_stripe.stl
- added link left_thigh_stripe, mass 0.05; collision box size=0.004525 0.037827 0.182634; visual mesh filename=package://iron_man_mark_43/meshes/left_thigh_stripe.stl
- added link neck_ring, mass 0.3; collision box size=0.16 0.16 0.025; visual mesh filename=package://iron_man_mark_43/meshes/neck_ring.stl
- added link right_gauntlet_stripe, mass 0.03; collision box size=0.004853 0.032695 0.102794; visual mesh filename=package://iron_man_mark_43/meshes/right_gauntlet_stripe.stl
- added link right_shin_stripe, mass 0.05; collision box size=0.005233 0.042669 0.162674; visual mesh filename=package://iron_man_mark_43/meshes/right_shin_stripe.stl
- added link right_thigh_stripe, mass 0.05; collision box size=0.004525 0.037827 0.182634; visual mesh filename=package://iron_man_mark_43/meshes/right_thigh_stripe.stl
- link left_bicep_clamshell: geometry collision box size=0.119616 0.039871 0.228308; visual mesh filename=package://iron_man_mark_43/meshes/left_bicep_clamshell.stl
- link left_bicep_sleeve: geometry collision box size=0.15959 0.15171 0.228306; visual mesh filename=package://iron_man_mark_43/meshes/left_bicep_sleeve.stl
- link left_calf_clamshell: geometry collision box size=0.154507 0.055798 0.327702; visual mesh filename=package://iron_man_mark_43/meshes/left_calf_clamshell.stl
- link left_chest_door: geometry collision box size=0.134852 0.240172 0.34; visual mesh filename=package://iron_man_mark_43/meshes/left_chest_door.stl
- link left_elbow_cap: geometry collision box size=0.117867 0.117867 0.043982; visual mesh filename=package://iron_man_mark_43/meshes/left_elbow_cap.stl
- link left_gauntlet_clamshell: geometry collision box size=0.105395 0.037654 0.189534; visual mesh filename=package://iron_man_mark_43/meshes/left_gauntlet_clamshell.s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
- link left_gauntlet_sleeve: geometry collision box size=0.14163 0.134065 0.189532; visual mesh filename=package://iron_man_mark_43/meshes/left_gauntlet_sleeve.stl
- link left_knee_cap: geometry collision box size=0.149828 0.149828 0.054978; visual mesh filename=package://iron_man_mark_43/meshes/left_knee_cap.stl
- link left_pauldron: geometry collision box size=0.269818 0.269818 0.094979; visual mesh filename=package://iron_man_mark_43/meshes/left_pauldron.stl
- link left_pauldron_edge: geometry collision box size=0.012145 0.091966 0.033932; visual mesh filename=package://iron_man_mark_43/meshes/left_pauldron_edge.stl
- link left_shin_shell: geometry collision box size=0.207453 0.196274 0.3277; visual mesh filename=package://iron_man_mark_43/meshes/left_shin_shell.stl
- link left_thigh_clamshell: geometry collision box size=0.180452 0.062313 0.343583; visual mesh filename=package://iron_man_mark_43/meshes/left_thigh_clamshell.stl
- link left_thigh_shell: geometry collision box size=0.241367 0.228928 0.343581; visual mesh filename=package://iron_man_mark_43/meshes/left_thigh_shell.stl
- link right_bicep_clamshell: geometry collision box size=0.119616 0.039871 0.228308; visual mesh filename=package://iron_man_mark_43/meshes/right_bicep_clamshell.stl
- link right_bicep_sleeve: geometry collision box size=0.15959 0.15171 0.228306; visual mesh filename=package://iron_man_mark_43/meshes/right_bicep_sleeve.stl
- link right_calf_clamshell: geometry collision box size=0.154506 0.055798 0.327702; visual mesh filename=package://iron_man_mark_43/meshes/right_calf_clamshell.stl
- link right_chest_door: geometry collision box size=0.134865 0.240172 0.34; visual mesh filename=package://iron_man_mark_43/meshes/right_chest_door.stl
- link right_elbow_cap: geometry collision box size=0.117867 0.117867 0.043982; visual mesh filename=package://iron_man_mark_43/meshes/right_elbow_cap.stl
- link right_gauntlet_clamshell: geometry collision box size=0.105394 0.037654 0.189534; visual mesh filename=package://iron_man_mark_43/meshes/right_gauntlet_clamshell.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
- link right_gauntlet_sleeve: geometry collision box size=0.14163 0.134065 0.189532; visual mesh filename=package://iron_man_mark_43/meshes/right_gauntlet_sleeve.stl
- link right_knee_cap: geometry collision box size=0.149828 0.149828 0.054978; visual mesh filename=package://iron_man_mark_43/meshes/right_knee_cap.stl
- link right_pauldron: geometry collision box size=0.269818 0.269818 0.094979; visual mesh filename=package://iron_man_mark_43/meshes/right_pauldron.stl
- link right_pauldron_edge: geometry collision box size=0.012145 0.091966 0.033932; visual mesh filename=package://iron_man_mark_43/meshes/right_pauldron_edge.stl
- link right_shin_shell: geometry collision box size=0.207454 0.196274 0.3277; visual mesh filename=package://iron_man_mark_43/meshes/right_shin_shell.stl
- link right_thigh_clamshell: geometry collision box size=0.180452 0.062313 0.343583; visual mesh filename=package://iron_man_mark_43/meshes/right_thigh_clamshell.stl
- link right_thigh_shell: geometry collision box size=0.241367 0.228928 0.343581; visual mesh filename=package://iron_man_mark_43/meshes/right_thigh_shell.stl
Joints:
- added joint left_gauntlet_stripe_mount: type fixed, parent left_gauntlet_sleeve, child left_gauntlet_stripe, origin xyz=0.067 0 -0.09 rpy=0 0 0
- added joint left_shin_stripe_mount: type fixed, parent left_shin_shell, child left_shin_stripe, origin xyz=0.099 0 -0.16 rpy=0 0 0
- added joint left_thigh_stripe_mount: type fixed, parent left_thigh_shell, child left_thigh_stripe, origin xyz=0 0.116 -0.17 rpy=0 0 1.570796
- added joint neck_ring_mount: type fixed, parent spine_frame, child neck_ring, origin xyz=0.02 0 0.524 rpy=0 0 0
- added joint right_gauntlet_stripe_mount: type fixed, parent right_gauntlet_sleeve, child right_gauntlet_stripe, origin xyz=0.067 0 -0.09 rpy=0 0 0
- added joint right_shin_stripe_mount: type fixed, parent right_shin_shell, child right_shin_stripe, origin xyz=0.099 0 -0.16 rpy=0 0 0
- added joint right_thigh_stripe_mount: type fixed, parent right_thigh_shell, child right_thigh_stripe, origin xyz=0 -0.116 -0.17 rpy=0 0 -1.570796
- joint left_bicep_clamshell_hinge: origin xyz=0.037318 -0.115057 -0.04557 rpy=0 0 0 -> xyz=0.037318 -0.115057 -0.03906 rpy=0 0 0
- joint left_bicep_sleeve_mount: origin xyz=0 -0.05 -0.04557 rpy=0 0 0 -> xyz=0 -0.05 -0.03906 rpy=0 0 0
- joint left_calf_clamshell_hinge: origin xyz=0.048762 -0.130007 -0.05166 rpy=0 0 0 -> xyz=0.048762 -0.130007 -0.04305 rpy=0 0 0
- joint left_gauntlet_clamshell_hinge: origin xyz=0.03284 -0.10225 -0.033215 rpy=0 0 0 -> xyz=0.03284 -0.10225 -0.028105 rpy=0 0 0
- joint left_gauntlet_sleeve_mount: origin xyz=0 -0.045 -0.033215 rpy=0 0 0 -> xyz=0 -0.045 -0.028105 rpy=0 0 0
- joint left_pauldron_edge_mount: origin xyz=0.117 0 0.022 rpy=0 0 0 -> xyz=0.127 0 0.024 rpy=0 0 0
- joint left_pauldron_hinge: origin xyz=0 -0.02 0.025 rpy=-0.45 0 0 -> xyz=0 -0.02 0.02 rpy=-0.45 0 0
- joint left_shin_shell_mount: origin xyz=0 -0.045 -0.05166 rpy=0 0 0 -> xyz=0 -0.045 -0.04305 rpy=0 0 0
- joint left_thigh_clamshell_hinge: origin xyz=0.057221 -0.144754 -0.05145 rpy=0 0 0 -> xyz=0.057221 -0.144754 -0.042875 rpy=0 0 0
- joint left_thigh_shell_mount: origin xyz=0 -0.045 -0.05145 rpy=0 0 0 -> xyz=0 -0.045 -0.042875 rpy=0 0 0
- joint right_bicep_clamshell_hinge: origin xyz=0.037318 0.115057 -0.04557 rpy=0 0 0 -> xyz=0.037318 0.115057 -0.03906 rpy=0 0 0
- joint right_bicep_sleeve_mount: origin xyz=0 0.05 -0.04557 rpy=0 0 0 -> xyz=0 0.05 -0.03906 rpy=0 0 0
- joint right_calf_clamshell_hinge: origin xyz=0.048762 0.130007 -0.05166 rpy=0 0 0 -> xyz=0.048762 0.130007 -0.04305 rpy=0 0 0
- joint right_gauntlet_clamshell_hinge: origin xyz=0.03284 0.10225 -0.033215 rpy=0 0 0 -> xyz=0.03284 0.10225 -0.028105 rpy=0 0 0
- joint right_gauntlet_sleeve_mount: origin xyz=0 0.045 -0.033215 rpy=0 0 0 -> xyz=0 0.045 -0.028105 rpy=0 0 0
- joint right_pauldron_edge_mount: origin xyz=0.117 0 0.022 rpy=0 0 0 -> xyz=0.127 0 0.024 rpy=0 0 0
- joint right_pauldron_hinge: origin xyz=0 0.02 0.025 rpy=0.45 0 0 -> xyz=0 0.02 0.02 rpy=0.45 0 0
- joint right_shin_shell_mount: origin xyz=0 0.045 -0.05166 rpy=0 0 0 -> xyz=0 0.045 -0.04305 rpy=0 0 0
- joint right_thigh_clamshell_hinge: origin xyz=0.057221 0.144754 -0.05145 rpy=0 0 0 -> xyz=0.057221 0.144754 -0.042875 rpy=0 0 0
- joint right_thigh_shell_mount: origin xyz=0 0.045 -0.05145 rpy=0 0 0 -> xyz=0 0.045 -0.042875 rpy=0 0 0

Commit message: Fix physical model fidelity and add dimensioned solid CAD enclosures

File: examples/14_iron_man_mark_43/robot.sim.urdf (robot description, URDF)
Before this commit: robot iron_man_mark_43, 132 links, 131 joints
Links:
- link left_boot_toe: geometry collision box size=0.077945 0.129908 0.064957; visual mesh filename=meshes/left_boot_toe.stl
- link right_boot_toe: geometry collision box size=0.077945 0.129908 0.064957; visual mesh filename=meshes/right_boot_toe.stl

File: examples/14_iron_man_mark_43/robot.urdf (robot description, URDF)
Before this commit: robot iron_man_mark_43, 132 links, 131 joints
Links:
- link left_boot_toe: geometry collision box size=0.077945 0.129908 0.064957; visual mesh filename=package://iron_man_mark_43/meshes/left_boot_toe.stl
- link right_boot_toe: geometry collision box size=0.077945 0.129908 0.064957; visual mesh filename=package://iron_man_mark_43/meshes/right_boot_toe.stl
