Commit message: Repair solid geometry and integrate dimensioned CAD with audited collision exports

File: examples/14_iron_man_mark_43/robot.urdf (robot description, URDF)
Before this commit: robot iron_man_mark_43, 132 links, 131 joints
Links:
- link ab_plate_1: geometry collision box size=0.037696 0.223034 0.04492; visual mesh filename=package://iron_man_mark_43/meshes/ab_plate_1.stl
- link ab_plate_2: geometry collision box size=0.032497 0.206461 0.04492; visual mesh filename=package://iron_man_mark_43/meshes/ab_plate_2.stl
- link ab_plate_3: geometry collision box size=0.027716 0.189373 0.04492; visual mesh filename=package://iron_man_mark_43/meshes/ab_plate_3.stl
- link back_shell: geometry collision box size=0.043788 0.366351 0.459092; visual mesh filename=package://iron_man_mark_43/meshes/back_shell.stl
- link belt_plate: geometry collision box size=0.041001 0.40942 0.099812; visual mesh filename=package://iron_man_mark_43/meshes/belt_plate.stl
- link chest_centre: geometry collision box size=0.011869 0.158703 0.199612; visual mesh filename=package://iron_man_mark_43/meshes/chest_centre.stl
- link codpiece: geometry collision box size=0.01798 0.122986 0.139732; visual mesh filename=package://iron_man_mark_43/meshes/codpiece.stl
- link collar_plate: geometry collision box size=0.055374 0.334683 0.089832; visual mesh filename=package://iron_man_mark_43/meshes/collar_plate.stl
- link helmet: geometry collision box size=0.124457 0.204 0.205; visual mesh filename=package://iron_man_mark_43/meshes/helmet_cranium.stl
- link helmet_crown_panel: geometry collision box size=0.116457 0.174 0.045818; visual mesh filename=package://iron_man_mark_43/meshes/helmet_crown_panel.stl
- link left_ankle_flap: geometry collision box size=0.008608 0.057139 0.079848; visual mesh filename=package://iron_man_mark_43/meshes/left_ankle_flap.stl
- link left_bicep_clamshell: geometry collision box size=0.113161 0.037217 0.227874; visual mesh filename=package://iron_man_mark_43/meshes/left_bicep_clamshell.stl
- link left_bicep_sleeve: geometry collision box size=0.14959 0.142475 0.227874; visual mesh filename=package://iron_man_mark_43/meshes/left_bicep_sleeve.stl
- link left_boot_toe: geometry collision box size=0.072 0.12 0.060652; visual mesh filename=package://iron_man_mark_43/meshes/left_boot_toe.stl
- link left_boot_trim: geometry collision box size=0.013892 0.095108 0.07985; visual mesh filename=package://iron_man_mark_43/meshes/left_boot_trim.stl
- link left_calf_clamshell: geometry collision box size=0.146769 0.05262 0.327465; visual mesh filename=package://iron_man_mark_43/meshes/left_calf_clamshell.stl
- link left_chest_door: geometry collision box size=0.102277 0.223424 0.3; visual mesh filename=package://iron_man_mark_43/meshes/left_chest_door.stl
- link left_elbow_cap: geometry collision box size=0.11 0.11 0.040712; visual mesh filename=package://iron_man_mark_43/meshes/left_elbow_cap.stl
- link left_eye_lens: geometry collision box size=0.025208 0.049 0.021; visual mesh filename=package://iron_man_mark_43/meshes/helmet_left_eye_lens.stl
- link left_eye_socket: geometry collision box size=0.042726 0.059 0.029; visual mesh filename=package://iron_man_mark_43/meshes/helmet_left_eye_socket.stl
- link left_finger_1: geometry collision box size=0.012009 0.013888 0.059896; visual mesh filename=package://iron_man_mark_43/meshes/left_finger_1.stl
- link left_finger_2: geometry collision box size=0.012009 0.013888 0.059896; visual mesh filename=package://iron_man_mark_43/meshes/left_finger_2.stl
- link left_finger_3: geometry collision box size=0.012009 0.013888 0.059896; visual mesh filename=package://iron_man_mark_43/meshes/left_finger_3.stl
- link left_finger_4: geometry collision box size=0.012009 0.013888 0.059896; visual mesh filename=package://iron_man_mark_43/meshes/left_finger_4.stl
- link left_flight_flap: geometry collision box size=0.007278 0.118321 0.179648; visual mesh filename=package://iron_man_mark_43/meshes/left_flight_flap.stl
- link left_forearm_cuff: geometry collision box size=0.1 0.1 0.06; visual mesh filename=package://iron_man_mark_43/meshes/left_forearm_cuff.stl
- link left_gauntlet_clamshell: geometry collision box size=0.098947 0.035004 0.189304; visual mesh filename=package://iron_man_mark_43/meshes/left_gauntlet_clamshell.s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
- link left_gauntlet_hatch: geometry collision box size=0.005992 0.043281 0.039926; visual mesh filename=package://iron_man_mark_43/meshes/left_gauntlet_hatch.stl
- link left_gauntlet_sleeve: geometry collision box size=0.13164 0.124839 0.189303; visual mesh filename=package://iron_man_mark_43/meshes/left_gauntlet_sleeve.stl
- link left_gauntlet_stripe: geometry collision box size=0.004242 0.029133 0.099806; visual mesh filename=package://iron_man_mark_43/meshes/left_gauntlet_stripe.stl
- link left_hand_plate: geometry collision box size=0.010482 0.066353 0.09981; visual mesh filename=package://iron_man_mark_43/meshes/left_hand_plate.stl
- link left_hip_flap: geometry collision box size=0.017752 0.133455 0.149712; visual mesh filename=package://iron_man_mark_43/meshes/left_hip_flap.stl
- link left_knee_cap: geometry collision box size=0.13 0.13 0.026618; visual mesh filename=package://iron_man_mark_43/meshes/left_knee_cap.stl
- link left_lat_plate: geometry collision box size=0.043257 0.345798 0.23953; visual mesh filename=package://iron_man_mark_43/meshes/left_lat_plate.stl
- link left_pauldron: geometry collision box size=0.22 0.22 0.066087; visual mesh filename=package://iron_man_mark_43/meshes/left_pauldron.stl
- link left_pauldron_edge: geometry collision box size=0.01083 0.086856 0.029948; visual mesh filename=package://iron_man_mark_43/meshes/left_pauldron_edge.stl
- link left_pectoral_trim: geometry collision box size=0.005285 0.059522 0.109788; visual mesh filename=package://iron_man_mark_43/meshes/left_pectoral_trim.stl
- link left_shank_cuff: geometry collision box size=0.146 0.146 0.07; visual mesh filename=package://iron_man_mark_43/meshes/left_shank_cuff.stl
- link left_shin_guard: geometry collision box size=0.015517 0.093488 0.09981; visual mesh filename=package://iron_man_mark_43/meshes/left_shin_guard.stl
- link left_shin_shell: geometry collision box size=0.195465 0.185203 0.327464; visual mesh filename=package://iron_man_mark_43/meshes/left_shin_shell.stl
- link left_shin_stripe: geometry collision box size=0.007624 0.062904 0.064876; visual mesh filename=package://iron_man_mark_43/meshes/left_shin_stripe.stl
- link left_thigh_clamshell: geometry collision box size=0.17271 0.059129 0.343186; visual mesh filename=package://iron_man_mark_43/meshes/left_thigh_clamshell.stl
- link left_thigh_cuff: geometry collision box size=0.18 0.18 0.07; visual mesh filename=package://iron_man_mark_43/meshes/left_thigh_cuff.stl
- link left_thigh_shell: geometry collision box size=0.229372 0.217851 0.343185; visual mesh filename=package://iron_man_mark_43/meshes/left_thigh_shell.stl
- link left_thigh_stripe: geometry collision box size=0.009983 0.081737 0.209586; visual mesh filename=package://iron_man_mark_43/meshes/left_thigh_stripe.stl
- link left_thruster_cover: geometry collision box size=0.010848 0.076326 0.069868; visual mesh filename=package://iron_man_mark_43/meshes/left_thruster_cover.stl
- link left_thumb: geometry collision box size=0.012009 0.013888 0.049916; visual mesh filename=package://iron_man_mark_43/meshes/left_thumb.stl
- link left_upper_arm_cuff: geometry collision box size=0.12 0.12 0.06; visual mesh filename=package://iron_man_mark_43/meshes/left_upper_arm_cuff.stl
- link mouth_line: geometry collision box size=0.01731 0.096109 0.005; visual mesh filename=package://iron_man_mark_43/meshes/helmet_mouth_line.stl
- link pelvis_frame: geometry collision box size=0.22 0.34 0.09; visual mesh filename=package://iron_man_mark_43/meshes/pelvis_frame.stl
- link rear_belt_plate: geometry collision box size=0.041001 0.40942 0.099812; visual mesh filename=package://iron_man_mark_43/meshes/rear_belt_plate.stl
- link right_ankle_flap: geometry collision box size=0.008608 0.057139 0.079848; visual mesh filename=package://iron_man_mark_43/meshes/right_ankle_flap.stl
- link right_bicep_clamshell: geometry collision box size=0.113161 0.037217 0.227874; visual mesh filename=package://iron_man_mark_43/meshes/right_bicep_clamshell.stl
- link right_bicep_sleeve: geometry collision box size=0.14959 0.142475 0.227874; visual mesh filename=package://iron_man_mark_43/meshes/right_bicep_sleeve.stl
- link right_boot_toe: geometry collision box size=0.072 0.12 0.060652; visual mesh filename=package://iron_man_mark_43/meshes/right_boot_toe.stl
- link right_boot_trim: geometry collision box size=0.013892 0.095108 0.07985; visual mesh filename=package://iron_man_mark_43/meshes/right_boot_trim.stl
- link right_calf_clamshell: geometry collision box size=0.146769 0.05262 0.327465; visual mesh filename=package://iron_man_mark_43/meshes/right_calf_clamshell.stl
- link right_chest_door: geometry collision box size=0.10227 0.223424 0.3; visual mesh filename=package://iron_man_mark_43/meshes/right_chest_door.stl
- link right_elbow_cap: geometry collision box size=0.11 0.11 0.040712; visual mesh filename=package://iron_man_mark_43/meshes/right_elbow_cap.stl
- link right_eye_lens: geometry collision box size=0.025208 0.049 0.021; visual mesh filename=package://iron_man_mark_43/meshes/helmet_right_eye_lens.stl
- link right_eye_socket: geometry collision box size=0.042726 0.059 0.029; visual mesh filename=package://iron_man_mark_43/meshes/helmet_right_eye_socket.s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
- link right_finger_1: geometry collision box size=0.012009 0.013888 0.059896; visual mesh filename=package://iron_man_mark_43/meshes/right_finger_1.stl
- link right_finger_2: geometry collision box size=0.012009 0.013888 0.059896; visual mesh filename=package://iron_man_mark_43/meshes/right_finger_2.stl
- link right_finger_3: geometry collision box size=0.012009 0.013888 0.059896; visual mesh filename=package://iron_man_mark_43/meshes/right_finger_3.stl
- link right_finger_4: geometry collision box size=0.012009 0.013888 0.059896; visual mesh filename=package://iron_man_mark_43/meshes/right_finger_4.stl
- link right_flight_flap: geometry collision box size=0.007278 0.118321 0.179648; visual mesh filename=package://iron_man_mark_43/meshes/right_flight_flap.stl
- link right_forearm_cuff: geometry collision box size=0.1 0.1 0.06; visual mesh filename=package://iron_man_mark_43/meshes/right_forearm_cuff.stl
- link right_gauntlet_clamshell: geometry collision box size=0.098947 0.035004 0.189304; visual mesh filename=package://iron_man_mark_43/meshes/right_gauntlet_clamshell.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
- link right_gauntlet_hatch: geometry collision box size=0.005992 0.043281 0.039926; visual mesh filename=package://iron_man_mark_43/meshes/right_gauntlet_hatch.stl
- link right_gauntlet_sleeve: geometry collision box size=0.13164 0.124839 0.189303; visual mesh filename=package://iron_man_mark_43/meshes/right_gauntlet_sleeve.stl
- link right_gauntlet_stripe: geometry collision box size=0.004242 0.029133 0.099806; visual mesh filename=package://iron_man_mark_43/meshes/right_gauntlet_stripe.stl
- link right_hand_plate: geometry collision box size=0.010482 0.066353 0.09981; visual mesh filename=package://iron_man_mark_43/meshes/right_hand_plate.stl
- link right_hip_flap: geometry collision box size=0.017752 0.133455 0.149712; visual mesh filename=package://iron_man_mark_43/meshes/right_hip_flap.stl
- link right_knee_cap: geometry collision box size=0.13 0.13 0.026618; visual mesh filename=package://iron_man_mark_43/meshes/right_knee_cap.stl
- link right_lat_plate: geometry collision box size=0.043257 0.345798 0.23953; visual mesh filename=package://iron_man_mark_43/meshes/right_lat_plate.stl
- link right_pauldron: geometry collision box size=0.22 0.22 0.066087; visual mesh filename=package://iron_man_mark_43/meshes/right_pauldron.stl
- link right_pauldron_edge: geometry collision box size=0.01083 0.086856 0.029948; visual mesh filename=package://iron_man_mark_43/meshes/right_pauldron_edge.stl
- link right_pectoral_trim: geometry collision box size=0.005285 0.059522 0.109788; visual mesh filename=package://iron_man_mark_43/meshes/right_pectoral_trim.stl
- link right_shank_cuff: geometry collision box size=0.146 0.146 0.07; visual mesh filename=package://iron_man_mark_43/meshes/right_shank_cuff.stl
- link right_shin_guard: geometry collision box size=0.015517 0.093488 0.09981; visual mesh filename=package://iron_man_mark_43/meshes/right_shin_guard.stl
- link right_shin_shell: geometry collision box size=0.195465 0.185203 0.327464; visual mesh filename=package://iron_man_mark_43/meshes/right_shin_shell.stl
- link right_shin_stripe: geometry collision box size=0.007624 0.062904 0.064876; visual mesh filename=package://iron_man_mark_43/meshes/right_shin_stripe.stl
- link right_thigh_clamshell: geometry collision box size=0.17271 0.059129 0.343186; visual mesh filename=package://iron_man_mark_43/meshes/right_thigh_clamshell.stl
- link right_thigh_cuff: geometry collision box size=0.18 0.18 0.07; visual mesh filename=package://iron_man_mark_43/meshes/right_thigh_cuff.stl
- link right_thigh_shell: geometry collision box size=0.229372 0.217851 0.343185; visual mesh filename=package://iron_man_mark_43/meshes/right_thigh_shell.stl
- link right_thigh_stripe: geometry collision box size=0.009983 0.081737 0.209586; visual mesh filename=package://iron_man_mark_43/meshes/right_thigh_stripe.stl
- link right_thruster_cover: geometry collision box size=0.010848 0.076326 0.069868; visual mesh filename=package://iron_man_mark_43/meshes/right_thruster_cover.stl
- link right_thumb: geometry collision box size=0.012009 0.013888 0.049916; visual mesh filename=package://iron_man_mark_43/meshes/right_thumb.stl
- link right_upper_arm_cuff: geometry collision box size=0.12 0.12 0.06; visual mesh filename=package://iron_man_mark_43/meshes/right_upper_arm_cuff.stl
Joints:
- joint left_ankle_flap_hinge: origin xyz=0 0.03 0.02 rpy=0 0 1.570796 -> xyz=0 0.085 0.02 rpy=0 0 1.570796
- joint left_hip_abduction: origin xyz=0 0.13 0.96425 rpy=0 0 0 -> xyz=0 0.17 0.96425 rpy=0 0 0
- joint left_hip_flap_hinge: origin xyz=0 0.2 1.03925 rpy=0 0 1.570796 -> xyz=0 0.275 1.03925 rpy=0 0 1.570796
- joint left_pauldron_edge_mount: origin xyz=0.127 0 0.024 rpy=0 0 0 -> xyz=0.107 0 0.024 rpy=0 0 0
- joint left_shin_stripe_mount: origin xyz=0.099 0 -0.16 rpy=0 0 0 -> xyz=0.099 0 -0.075 rpy=0 0 0
- joint left_shoulder_abduction: limit lower=-0.3 upper=2.6 effort=60 velocity=3 -> lower=-0.75 upper=2.15 effort=60 velocity=3; origin xyz=0 0.235 0 rpy=0 0 0 -> xyz=0 0.235 0 rpy=0.45 0 0
- joint left_thigh_stripe_mount: origin xyz=0 0.116 -0.17 rpy=0 0 1.570796 -> xyz=0.116 0 -0.15 rpy=0 0 0
- joint left_thumb_hinge: origin xyz=0.035 -0.085 -0.03 rpy=0 -1.570796 -0.8 -> xyz=0.035 -0.103 -0.03 rpy=0 -1.570796 -0.8
- joint right_ankle_flap_hinge: origin xyz=0 -0.03 0.02 rpy=0 0 -1.570796 -> xyz=0 -0.085 0.02 rpy=0 0 -1.570796
- joint right_hip_abduction: axis 1 0 0 -> -1 0 0; origin xyz=0 -0.13 0.96425 rpy=0 0 0 -> xyz=0 -0.17 0.96425 rpy=0 0 0
- joint right_hip_flap_hinge: origin xyz=0 -0.2 1.03925 rpy=0 0 -1.570796 -> xyz=0 -0.275 1.03925 rpy=0 0 -1.570796
- joint right_pauldron_edge_mount: origin xyz=0.127 0 0.024 rpy=0 0 0 -> xyz=0.107 0 0.024 rpy=0 0 0
- joint right_shin_stripe_mount: origin xyz=0.099 0 -0.16 rpy=0 0 0 -> xyz=0.099 0 -0.075 rpy=0 0 0
- joint right_shoulder_abduction: axis 1 0 0 -> -1 0 0; limit lower=-0.3 upper=2.6 effort=60 velocity=3 -> lower=-0.75 upper=2.15 effort=60 velocity=3; origin xyz=0 -0.235 0 rpy=0 0 0 -> xyz=0 -0.235 0 rpy=-0.45 0 0
- joint right_thigh_stripe_mount: origin xyz=0 -0.116 -0.17 rpy=0 0 -1.570796 -> xyz=0.116 0 -0.15 rpy=0 0 0
- joint right_thumb_hinge: origin xyz=0.035 0.085 -0.03 rpy=0 -1.570796 0.8 -> xyz=0.035 0.103 -0.03 rpy=0 -1.570796 0.8

Commit message: Reduce armour interference and validate tracking across joint trajectories

File: examples/14_iron_man_mark_43/robot.sim.urdf (robot description, URDF)
Before this commit: robot iron_man_mark_43, 132 links, 131 joints
Links:
- link left_lat_plate: geometry collision box size=0.031552 0.291187 0.17965; visual mesh filename=meshes/left_lat_plate.stl
- link right_lat_plate: geometry collision box size=0.031552 0.291187 0.17965; visual mesh filename=meshes/right_lat_plate.stl
Joints:
- joint left_lat_plate_hinge: origin xyz=-0.27 0.205 0.3024 rpy=0 0 1.570796 -> xyz=-0.27 0.185 0.2674 rpy=0 0 1.570796
- joint left_pauldron_hinge: origin xyz=0 -0.02 0.02 rpy=-0.45 0 0 -> xyz=0 0.025 0.065 rpy=-0.45 0 0
- joint right_lat_plate_hinge: origin xyz=-0.27 -0.205 0.3024 rpy=0 0 -1.570796 -> xyz=-0.27 -0.185 0.2674 rpy=0 0 -1.570796
- joint right_pauldron_hinge: origin xyz=0 0.02 0.02 rpy=0.45 0 0 -> xyz=0 -0.025 0.065 rpy=0.45 0 0

File: examples/14_iron_man_mark_43/robot.urdf (robot description, URDF)
Before this commit: robot iron_man_mark_43, 132 links, 131 joints
Links:
- link left_lat_plate: geometry collision box size=0.031552 0.291187 0.17965; visual mesh filename=package://iron_man_mark_43/meshes/left_lat_plate.stl
- link right_lat_plate: geometry collision box size=0.031552 0.291187 0.17965; visual mesh filename=package://iron_man_mark_43/meshes/right_lat_plate.stl
Joints:
- joint left_lat_plate_hinge: origin xyz=-0.27 0.205 0.3024 rpy=0 0 1.570796 -> xyz=-0.27 0.185 0.2674 rpy=0 0 1.570796
- joint left_pauldron_hinge: origin xyz=0 -0.02 0.02 rpy=-0.45 0 0 -> xyz=0 0.025 0.065 rpy=-0.45 0 0
- joint right_lat_plate_hinge: origin xyz=-0.27 -0.205 0.3024 rpy=0 0 -1.570796 -> xyz=-0.27 -0.185 0.2674 rpy=0 0 -1.570796
- joint right_pauldron_hinge: origin xyz=0 0.02 0.02 rpy=0.45 0 0 -> xyz=0 -0.025 0.065 rpy=0.45 0 0
