Commit message: Persist Mark 43 references and iterate curved torso and helmet surfaces

File: examples/14_iron_man_mark_43/robot.sim.urdf (robot description, URDF)
Before this commit: robot iron_man_mark_43, 238 links, 237 joints
Links:
- added link left_chest_inlay_centre, mass 0.06; collision box size=0.005162 0.074281 0.13; visual mesh filename=meshes/left_chest_inlay_centre.stl
- added link right_chest_inlay_centre, mass 0.06; collision box size=0.005162 0.074281 0.13; visual mesh filename=meshes/right_chest_inlay_centre.stl
- link chest_centre: geometry collision box size=0.007341 0.094573 0.22; visual mesh filename=meshes/chest_centre.stl
- link faceplate: geometry collision box size=0.051105 0.158461 0.206; visual mesh filename=meshes/helmet_faceplate.stl
- link forehead_plate: geometry collision box size=0.022294 0.08 0.021876; visual mesh filename=meshes/helmet_forehead_plate.stl
- link left_cheek_panel: geometry collision box size=0.150485 0.069259 0.206; visual mesh filename=meshes/helmet_left_cheek_panel.stl
- link left_chest_door: geometry collision box size=0.146661 0.233045 0.25823; visual mesh filename=meshes/left_chest_door.stl
- link left_chest_inlay: geometry collision box size=0.008624 0.108165 0.175; visual mesh filename=meshes/left_chest_inlay.stl
- link left_eye_lens: geometry collision box size=0.011362 0.049 0.014; visual mesh filename=meshes/helmet_left_eye_lens.stl
- link left_eye_socket: geometry collision box size=0.0216 0.059 0.029; visual mesh filename=meshes/helmet_left_eye_socket.stl
- link left_lat_plate: geometry collision box size=0.262367 0.125605 0.4; visual mesh filename=meshes/left_lat_plate.stl
- link left_pectoral_trim: mass 0.1 -> 0.25; geometry collision box size=0.142047 0.215998 0.097941; visual mesh filename=meshes/left_pectoral_trim.stl
- link left_rib_0: geometry collision box size=0.007012 0.103977 0.054; visual mesh filename=meshes/left_rib_0.stl
- link left_rib_1: geometry collision box size=0.007012 0.103977 0.054; visual mesh filename=meshes/left_rib_1.stl
- link left_rib_2: geometry collision box size=0.007012 0.103977 0.054; visual mesh filename=meshes/left_rib_2.stl
- link left_rib_edge_0: geometry collision box size=0.004572 0.085456 0.041; visual mesh filename=meshes/left_rib_edge_0.stl
- link left_rib_edge_1: geometry collision box size=0.004572 0.085456 0.041; visual mesh filename=meshes/left_rib_edge_1.stl
- link left_rib_edge_2: geometry collision box size=0.004572 0.085456 0.041; visual mesh filename=meshes/left_rib_edge_2.stl
- link left_rib_insert_0: geometry collision box size=0.003248 0.066705 0.027; visual mesh filename=meshes/left_rib_insert_0.stl
- link left_rib_insert_1: geometry collision box size=0.003248 0.066705 0.027; visual mesh filename=meshes/left_rib_insert_1.stl
- link left_rib_insert_2: geometry collision box size=0.003248 0.066705 0.027; visual mesh filename=meshes/left_rib_insert_2.stl
- link mouth_line: geometry collision box size=0.010014 0.08 0.003665; visual mesh filename=meshes/helmet_mouth_line.stl
- link right_cheek_panel: geometry collision box size=0.150485 0.069259 0.206; visual mesh filename=meshes/helmet_right_cheek_panel.stl
- link right_chest_door: geometry collision box size=0.149975 0.237603 0.264258; visual mesh filename=meshes/right_chest_door.stl
- link right_chest_inlay: geometry collision box size=0.008624 0.108165 0.175; visual mesh filename=meshes/right_chest_inlay.stl
- link right_eye_lens: geometry collision box size=0.011362 0.049 0.014; visual mesh filename=meshes/helmet_right_eye_lens.stl
- link right_eye_socket: geometry collision box size=0.0216 0.059 0.029; visual mesh filename=meshes/helmet_right_eye_socket.stl
- link right_lat_plate: geometry collision box size=0.262367 0.125583 0.4; visual mesh filename=meshes/right_lat_plate.stl
- link right_pectoral_trim: mass 0.1 -> 0.25; geometry collision box size=0.145571 0.22041 0.098558; visual mesh filename=meshes/right_pectoral_trim.stl
- link right_rib_0: geometry collision box size=0.007012 0.103977 0.054; visual mesh filename=meshes/right_rib_0.stl
- link right_rib_1: geometry collision box size=0.007012 0.103977 0.054; visual mesh filename=meshes/right_rib_1.stl
- link right_rib_2: geometry collision box size=0.007012 0.103977 0.054; visual mesh filename=meshes/right_rib_2.stl
- link right_rib_edge_0: geometry collision box size=0.004572 0.085456 0.041; visual mesh filename=meshes/right_rib_edge_0.stl
- link right_rib_edge_1: geometry collision box size=0.004572 0.085456 0.041; visual mesh filename=meshes/right_rib_edge_1.stl
- link right_rib_edge_2: geometry collision box size=0.004572 0.085456 0.041; visual mesh filename=meshes/right_rib_edge_2.stl
- link right_rib_insert_0: geometry collision box size=0.003248 0.066705 0.027; visual mesh filename=meshes/right_rib_insert_0.stl
- link right_rib_insert_1: geometry collision box size=0.003248 0.066705 0.027; visual mesh filename=meshes/right_rib_insert_1.stl
- link right_rib_insert_2: geometry collision box size=0.003248 0.066705 0.027; visual mesh filename=meshes/right_rib_insert_2.stl
Joints:
- added joint left_chest_inlay_centre_mount: type fixed, parent spine_frame, child left_chest_inlay_centre, origin xyz=0.174 0.16 0.33272 rpy=0 0 0.78
- added joint right_chest_inlay_centre_mount: type fixed, parent spine_frame, child right_chest_inlay_centre, origin xyz=0.174 -0.16 0.33272 rpy=0 0 -0.78
- joint chest_centre_mount: origin xyz=0.2 0 0.37772 rpy=0 0 0 -> xyz=0.204 0 0.37772 rpy=0 0 0
- joint left_chest_inlay_mount: origin xyz=0.15 0.178 0.33272 rpy=0 0 0.48 -> xyz=0.168 0.154 0.33272 rpy=0 0 0.78
- joint left_collar_inlay_mount: origin xyz=0.115 0.102 0.529 rpy=0 0 0 -> xyz=0.165 0.102 0.49 rpy=0 0 0
- joint left_lat_plate_fixed_knuckle_lower_mount: origin xyz=-0.27 0.185 0.30222 rpy=0 0 1.570796 -> xyz=-0.1 0.1 0.45722 rpy=0 0 0
- joint left_lat_plate_fixed_knuckle_upper_mount: origin xyz=-0.27 0.185 0.32322 rpy=0 0 1.570796 -> xyz=-0.1 0.1 0.47822 rpy=0 0 0
- joint left_lat_plate_hinge: origin xyz=-0.27 0.185 0.31272 rpy=0 0 1.570796 -> xyz=-0.1 0.1 0.46772 rpy=0 0 0
- joint left_pectoral_trim_mount: origin xyz=0.11 -0.132 0.078 rpy=0 0 0.18 -> xyz=-0.07 -0.24 0 rpy=0 0 0
- joint left_rib_0_mount: origin xyz=0.142 0.139 0.23 rpy=0 0.13 0.4 -> xyz=0.09 0.17 0.23 rpy=0 0.13 1.02
- joint left_rib_1_mount: origin xyz=0.133 0.129 0.165 rpy=0 0.13 0.4 -> xyz=0.084 0.161 0.165 rpy=0 0.13 1.02
- joint left_rib_2_mount: origin xyz=0.124 0.119 0.1 rpy=0 0.13 0.4 -> xyz=0.078 0.152 0.1 rpy=0 0.13 1.02
- joint left_rib_edge_0_mount: origin xyz=0.15 0.139 0.23 rpy=0 0.13 0.4 -> xyz=0.093 0.176 0.23 rpy=0 0.13 1.02
- joint left_rib_edge_1_mount: origin xyz=0.141 0.129 0.165 rpy=0 0.13 0.4 -> xyz=0.087 0.167 0.165 rpy=0 0.13 1.02
- joint left_rib_edge_2_mount: origin xyz=0.132 0.119 0.1 rpy=0 0.13 0.4 -> xyz=0.081 0.158 0.1 rpy=0 0.13 1.02
- joint left_rib_insert_0_mount: origin xyz=0.154 0.139 0.23 rpy=0 0.13 0.4 -> xyz=0.095 0.179 0.23 rpy=0 0.13 1.02
- joint left_rib_insert_1_mount: origin xyz=0.145 0.129 0.165 rpy=0 0.13 0.4 -> xyz=0.089 0.17 0.165 rpy=0 0.13 1.02
- joint left_rib_insert_2_mount: origin xyz=0.136 0.119 0.1 rpy=0 0.13 0.4 -> xyz=0.083 0.161 0.1 rpy=0 0.13 1.02
- joint right_chest_inlay_mount: origin xyz=0.15 -0.178 0.33272 rpy=0 0 -0.48 -> xyz=0.168 -0.154 0.33272 rpy=0 0 -0.78
- joint right_collar_inlay_mount: origin xyz=0.115 -0.102 0.529 rpy=0 0 0 -> xyz=0.165 -0.102 0.49 rpy=0 0 0
- joint right_lat_plate_fixed_knuckle_lower_mount: origin xyz=-0.27 -0.185 0.30222 rpy=0 0 -1.570796 -> xyz=-0.1 -0.1 0.45722 rpy=0 0 0
- joint right_lat_plate_fixed_knuckle_upper_mount: origin xyz=-0.27 -0.185 0.32322 rpy=0 0 -1.570796 -> xyz=-0.1 -0.1 0.47822 rpy=0 0 0
- joint right_lat_plate_hinge: origin xyz=-0.27 -0.185 0.31272 rpy=0 0 -1.570796 -> xyz=-0.1 -0.1 0.46772 rpy=0 0 0
- joint right_pectoral_trim_mount: origin xyz=0.11 0.132 0.078 rpy=0 0 -0.18 -> xyz=-0.07 0.24 0 rpy=0 0 0
- joint right_rib_0_mount: origin xyz=0.142 -0.139 0.23 rpy=0 -0.13 -0.4 -> xyz=0.09 -0.17 0.23 rpy=0 -0.13 -1.02
- joint right_rib_1_mount: origin xyz=0.133 -0.129 0.165 rpy=0 -0.13 -0.4 -> xyz=0.084 -0.161 0.165 rpy=0 -0.13 -1.02
- joint right_rib_2_mount: origin xyz=0.124 -0.119 0.1 rpy=0 -0.13 -0.4 -> xyz=0.078 -0.152 0.1 rpy=0 -0.13 -1.02
- joint right_rib_edge_0_mount: origin xyz=0.15 -0.139 0.23 rpy=0 -0.13 -0.4 -> xyz=0.093 -0.176 0.23 rpy=0 -0.13 -1.02
- joint right_rib_edge_1_mount: origin xyz=0.141 -0.129 0.165 rpy=0 -0.13 -0.4 -> xyz=0.087 -0.167 0.165 rpy=0 -0.13 -1.02
- joint right_rib_edge_2_mount: origin xyz=0.132 -0.119 0.1 rpy=0 -0.13 -0.4 -> xyz=0.081 -0.158 0.1 rpy=0 -0.13 -1.02
- joint right_rib_insert_0_mount: origin xyz=0.154 -0.139 0.23 rpy=0 -0.13 -0.4 -> xyz=0.095 -0.179 0.23 rpy=0 -0.13 -1.02
- joint right_rib_insert_1_mount: origin xyz=0.145 -0.129 0.165 rpy=0 -0.13 -0.4 -> xyz=0.089 -0.17 0.165 rpy=0 -0.13 -1.02
- joint right_rib_insert_2_mount: origin xyz=0.136 -0.119 0.1 rpy=0 -0.13 -0.4 -> xyz=0.083 -0.161 0.1 rpy=0 -0.13 -1.02

File: examples/14_iron_man_mark_43/robot.urdf (robot description, URDF)
Before this commit: robot iron_man_mark_43, 238 links, 237 joints
Links:
- added link left_chest_inlay_centre, mass 0.06; collision box size=0.005162 0.074281 0.13; visual mesh filename=package://iron_man_mark_43/meshes/left_chest_inlay_centre.s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
- added link right_chest_inlay_centre, mass 0.06; collision box size=0.005162 0.074281 0.13; visual mesh filename=package://iron_man_mark_43/meshes/right_chest_inlay_centre.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
- link chest_centre: geometry collision box size=0.007341 0.094573 0.22; visual mesh filename=package://iron_man_mark_43/meshes/chest_centre.stl
- link faceplate: geometry collision box size=0.051105 0.158461 0.206; visual mesh filename=package://iron_man_mark_43/meshes/helmet_faceplate.stl
- link forehead_plate: geometry collision box size=0.022294 0.08 0.021876; visual mesh filename=package://iron_man_mark_43/meshes/helmet_forehead_plate.stl
- link left_cheek_panel: geometry collision box size=0.150485 0.069259 0.206; visual mesh filename=package://iron_man_mark_43/meshes/helmet_left_cheek_panel.s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
- link left_chest_door: geometry collision box size=0.146661 0.233045 0.25823; visual mesh filename=package://iron_man_mark_43/meshes/left_chest_door.stl
- link left_chest_inlay: geometry collision box size=0.008624 0.108165 0.175; visual mesh filename=package://iron_man_mark_43/meshes/left_chest_inlay.stl
- link left_eye_lens: geometry collision box size=0.011362 0.049 0.014; visual mesh filename=package://iron_man_mark_43/meshes/helmet_left_eye_lens.stl
- link left_eye_socket: geometry collision box size=0.0216 0.059 0.029; visual mesh filename=package://iron_man_mark_43/meshes/helmet_left_eye_socket.stl
- link left_lat_plate: geometry collision box size=0.262367 0.125605 0.4; visual mesh filename=package://iron_man_mark_43/meshes/left_lat_plate.stl
- link left_pectoral_trim: mass 0.1 -> 0.25; geometry collision box size=0.142047 0.215998 0.097941; visual mesh filename=package://iron_man_mark_43/meshes/left_pectoral_trim.stl
- link left_rib_0: geometry collision box size=0.007012 0.103977 0.054; visual mesh filename=package://iron_man_mark_43/meshes/left_rib_0.stl
- link left_rib_1: geometry collision box size=0.007012 0.103977 0.054; visual mesh filename=package://iron_man_mark_43/meshes/left_rib_1.stl
- link left_rib_2: geometry collision box size=0.007012 0.103977 0.054; visual mesh filename=package://iron_man_mark_43/meshes/left_rib_2.stl
- link left_rib_edge_0: geometry collision box size=0.004572 0.085456 0.041; visual mesh filename=package://iron_man_mark_43/meshes/left_rib_edge_0.stl
- link left_rib_edge_1: geometry collision box size=0.004572 0.085456 0.041; visual mesh filename=package://iron_man_mark_43/meshes/left_rib_edge_1.stl
- link left_rib_edge_2: geometry collision box size=0.004572 0.085456 0.041; visual mesh filename=package://iron_man_mark_43/meshes/left_rib_edge_2.stl
- link left_rib_insert_0: geometry collision box size=0.003248 0.066705 0.027; visual mesh filename=package://iron_man_mark_43/meshes/left_rib_insert_0.stl
- link left_rib_insert_1: geometry collision box size=0.003248 0.066705 0.027; visual mesh filename=package://iron_man_mark_43/meshes/left_rib_insert_1.stl
- link left_rib_insert_2: geometry collision box size=0.003248 0.066705 0.027; visual mesh filename=package://iron_man_mark_43/meshes/left_rib_insert_2.stl
- link mouth_line: geometry collision box size=0.010014 0.08 0.003665; visual mesh filename=package://iron_man_mark_43/meshes/helmet_mouth_line.stl
- link right_cheek_panel: geometry collision box size=0.150485 0.069259 0.206; visual mesh filename=package://iron_man_mark_43/meshes/helmet_right_cheek_panel.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
- link right_chest_door: geometry collision box size=0.149975 0.237603 0.264258; visual mesh filename=package://iron_man_mark_43/meshes/right_chest_door.stl
- link right_chest_inlay: geometry collision box size=0.008624 0.108165 0.175; visual mesh filename=package://iron_man_mark_43/meshes/right_chest_inlay.stl
- link right_eye_lens: geometry collision box size=0.011362 0.049 0.014; visual mesh filename=package://iron_man_mark_43/meshes/helmet_right_eye_lens.stl
- link right_eye_socket: geometry collision box size=0.0216 0.059 0.029; visual mesh filename=package://iron_man_mark_43/meshes/helmet_right_eye_socket.s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
- link right_lat_plate: geometry collision box size=0.262367 0.125583 0.4; visual mesh filename=package://iron_man_mark_43/meshes/right_lat_plate.stl
- link right_pectoral_trim: mass 0.1 -> 0.25; geometry collision box size=0.145571 0.22041 0.098558; visual mesh filename=package://iron_man_mark_43/meshes/right_pectoral_trim.stl
- link right_rib_0: geometry collision box size=0.007012 0.103977 0.054; visual mesh filename=package://iron_man_mark_43/meshes/right_rib_0.stl
- link right_rib_1: geometry collision box size=0.007012 0.103977 0.054; visual mesh filename=package://iron_man_mark_43/meshes/right_rib_1.stl
- link right_rib_2: geometry collision box size=0.007012 0.103977 0.054; visual mesh filename=package://iron_man_mark_43/meshes/right_rib_2.stl
- link right_rib_edge_0: geometry collision box size=0.004572 0.085456 0.041; visual mesh filename=package://iron_man_mark_43/meshes/right_rib_edge_0.stl
- link right_rib_edge_1: geometry collision box size=0.004572 0.085456 0.041; visual mesh filename=package://iron_man_mark_43/meshes/right_rib_edge_1.stl
- link right_rib_edge_2: geometry collision box size=0.004572 0.085456 0.041; visual mesh filename=package://iron_man_mark_43/meshes/right_rib_edge_2.stl
- link right_rib_insert_0: geometry collision box size=0.003248 0.066705 0.027; visual mesh filename=package://iron_man_mark_43/meshes/right_rib_insert_0.stl
- link right_rib_insert_1: geometry collision box size=0.003248 0.066705 0.027; visual mesh filename=package://iron_man_mark_43/meshes/right_rib_insert_1.stl
- link right_rib_insert_2: geometry collision box size=0.003248 0.066705 0.027; visual mesh filename=package://iron_man_mark_43/meshes/right_rib_insert_2.stl
Joints:
- added joint left_chest_inlay_centre_mount: type fixed, parent spine_frame, child left_chest_inlay_centre, origin xyz=0.174 0.16 0.33272 rpy=0 0 0.78
- added joint right_chest_inlay_centre_mount: type fixed, parent spine_frame, child right_chest_inlay_centre, origin xyz=0.174 -0.16 0.33272 rpy=0 0 -0.78
- joint chest_centre_mount: origin xyz=0.2 0 0.37772 rpy=0 0 0 -> xyz=0.204 0 0.37772 rpy=0 0 0
- joint left_chest_inlay_mount: origin xyz=0.15 0.178 0.33272 rpy=0 0 0.48 -> xyz=0.168 0.154 0.33272 rpy=0 0 0.78
- joint left_collar_inlay_mount: origin xyz=0.115 0.102 0.529 rpy=0 0 0 -> xyz=0.165 0.102 0.49 rpy=0 0 0
- joint left_lat_plate_fixed_knuckle_lower_mount: origin xyz=-0.27 0.185 0.30222 rpy=0 0 1.570796 -> xyz=-0.1 0.1 0.45722 rpy=0 0 0
- joint left_lat_plate_fixed_knuckle_upper_mount: origin xyz=-0.27 0.185 0.32322 rpy=0 0 1.570796 -> xyz=-0.1 0.1 0.47822 rpy=0 0 0
- joint left_lat_plate_hinge: origin xyz=-0.27 0.185 0.31272 rpy=0 0 1.570796 -> xyz=-0.1 0.1 0.46772 rpy=0 0 0
- joint left_pectoral_trim_mount: origin xyz=0.11 -0.132 0.078 rpy=0 0 0.18 -> xyz=-0.07 -0.24 0 rpy=0 0 0
- joint left_rib_0_mount: origin xyz=0.142 0.139 0.23 rpy=0 0.13 0.4 -> xyz=0.09 0.17 0.23 rpy=0 0.13 1.02
- joint left_rib_1_mount: origin xyz=0.133 0.129 0.165 rpy=0 0.13 0.4 -> xyz=0.084 0.161 0.165 rpy=0 0.13 1.02
- joint left_rib_2_mount: origin xyz=0.124 0.119 0.1 rpy=0 0.13 0.4 -> xyz=0.078 0.152 0.1 rpy=0 0.13 1.02
- joint left_rib_edge_0_mount: origin xyz=0.15 0.139 0.23 rpy=0 0.13 0.4 -> xyz=0.093 0.176 0.23 rpy=0 0.13 1.02
- joint left_rib_edge_1_mount: origin xyz=0.141 0.129 0.165 rpy=0 0.13 0.4 -> xyz=0.087 0.167 0.165 rpy=0 0.13 1.02
- joint left_rib_edge_2_mount: origin xyz=0.132 0.119 0.1 rpy=0 0.13 0.4 -> xyz=0.081 0.158 0.1 rpy=0 0.13 1.02
- joint left_rib_insert_0_mount: origin xyz=0.154 0.139 0.23 rpy=0 0.13 0.4 -> xyz=0.095 0.179 0.23 rpy=0 0.13 1.02
- joint left_rib_insert_1_mount: origin xyz=0.145 0.129 0.165 rpy=0 0.13 0.4 -> xyz=0.089 0.17 0.165 rpy=0 0.13 1.02
- joint left_rib_insert_2_mount: origin xyz=0.136 0.119 0.1 rpy=0 0.13 0.4 -> xyz=0.083 0.161 0.1 rpy=0 0.13 1.02
- joint right_chest_inlay_mount: origin xyz=0.15 -0.178 0.33272 rpy=0 0 -0.48 -> xyz=0.168 -0.154 0.33272 rpy=0 0 -0.78
- joint right_collar_inlay_mount: origin xyz=0.115 -0.102 0.529 rpy=0 0 0 -> xyz=0.165 -0.102 0.49 rpy=0 0 0
- joint right_lat_plate_fixed_knuckle_lower_mount: origin xyz=-0.27 -0.185 0.30222 rpy=0 0 -1.570796 -> xyz=-0.1 -0.1 0.45722 rpy=0 0 0
- joint right_lat_plate_fixed_knuckle_upper_mount: origin xyz=-0.27 -0.185 0.32322 rpy=0 0 -1.570796 -> xyz=-0.1 -0.1 0.47822 rpy=0 0 0
- joint right_lat_plate_hinge: origin xyz=-0.27 -0.185 0.31272 rpy=0 0 -1.570796 -> xyz=-0.1 -0.1 0.46772 rpy=0 0 0
- joint right_pectoral_trim_mount: origin xyz=0.11 0.132 0.078 rpy=0 0 -0.18 -> xyz=-0.07 0.24 0 rpy=0 0 0
- joint right_rib_0_mount: origin xyz=0.142 -0.139 0.23 rpy=0 -0.13 -0.4 -> xyz=0.09 -0.17 0.23 rpy=0 -0.13 -1.02
- joint right_rib_1_mount: origin xyz=0.133 -0.129 0.165 rpy=0 -0.13 -0.4 -> xyz=0.084 -0.161 0.165 rpy=0 -0.13 -1.02
- joint right_rib_2_mount: origin xyz=0.124 -0.119 0.1 rpy=0 -0.13 -0.4 -> xyz=0.078 -0.152 0.1 rpy=0 -0.13 -1.02
- joint right_rib_edge_0_mount: origin xyz=0.15 -0.139 0.23 rpy=0 -0.13 -0.4 -> xyz=0.093 -0.176 0.23 rpy=0 -0.13 -1.02
- joint right_rib_edge_1_mount: origin xyz=0.141 -0.129 0.165 rpy=0 -0.13 -0.4 -> xyz=0.087 -0.167 0.165 rpy=0 -0.13 -1.02
- joint right_rib_edge_2_mount: origin xyz=0.132 -0.119 0.1 rpy=0 -0.13 -0.4 -> xyz=0.081 -0.158 0.1 rpy=0 -0.13 -1.02
- joint right_rib_insert_0_mount: origin xyz=0.154 -0.139 0.23 rpy=0 -0.13 -0.4 -> xyz=0.095 -0.179 0.23 rpy=0 -0.13 -1.02
- joint right_rib_insert_1_mount: origin xyz=0.145 -0.129 0.165 rpy=0 -0.13 -0.4 -> xyz=0.089 -0.17 0.165 rpy=0 -0.13 -1.02
- joint right_rib_insert_2_mount: origin xyz=0.136 -0.119 0.1 rpy=0 -0.13 -0.4 -> xyz=0.083 -0.161 0.1 rpy=0 -0.13 -1.02
