Commit message: Resolve torso, wrist, cuff and clamshell interference with reproducible surface audits

File: examples/14_iron_man_mark_43/robot.sim.urdf (robot description, URDF)
Before this commit: robot iron_man_mark_43, 268 links, 267 joints
Links:
- link ab_plate_3: geometry collision box size=0.018372 0.20326 0.043; visual mesh filename=meshes/ab_plate_3.stl
- link chest_plate: geometry collision box size=0.02 0.16 0.24; visual box size=0.02 0.16 0.24
- link left_bicep_clamshell: geometry collision box size=0.109834 0.043268 0.26691; visual mesh filename=meshes/left_bicep_clamshell.stl
- link left_bicep_front: geometry collision box size=0.017641 0.077505 0.202852; visual mesh filename=meshes/left_bicep_front.stl
- link left_bicep_sleeve: geometry collision box size=0.14967 0.138399 0.26691; visual mesh filename=meshes/left_bicep_sleeve.stl
- link left_calf_clamshell: geometry collision box size=0.135784 0.059588 0.37884; visual mesh filename=meshes/left_calf_clamshell.stl
- link left_chest_door: geometry collision box size=0.146048 0.233043 0.204085; visual mesh filename=meshes/left_chest_door.stl
- link left_forearm_crest: geometry collision box size=0.022191 0.090293 0.177828; visual mesh filename=meshes/left_forearm_crest.stl
- link left_gauntlet_clamshell: geometry collision box size=0.100056 0.043404 0.222285; visual mesh filename=meshes/left_gauntlet_clamshell.stl
- link left_gauntlet_sleeve: geometry collision box size=0.136346 0.125376 0.222285; visual mesh filename=meshes/left_gauntlet_sleeve.stl
- link left_hand: geometry collision box size=0.09 0.07 0.03; visual box size=0.09 0.07 0.03
- link left_hand_plate: geometry collision box size=0.014302 0.083899 0.08983; visual mesh filename=meshes/left_hand_plate.stl
- link left_hip_cowl: geometry collision box size=0.174356 0.174015 0.1; visual mesh filename=meshes/left_hip_cowl.stl
- link left_lat_plate: geometry collision box size=0.161485 0.101377 0.35; visual mesh filename=meshes/left_lat_plate.stl
- link left_pectoral_trim: geometry collision box size=0.142149 0.215993 0.07783; visual mesh filename=meshes/left_pectoral_trim.stl
- link left_shin_edge: geometry collision box size=0.018441 0.020286 0.2614; visual mesh filename=meshes/left_shin_edge.stl
- link left_shin_ridge: geometry collision box size=0.023159 0.051957 0.253823; visual mesh filename=meshes/left_shin_ridge.stl
- link left_shin_shell: geometry collision box size=0.185031 0.169954 0.37884; visual mesh filename=meshes/left_shin_shell.stl
- link left_shin_stripe: geometry collision box size=0.030225 0.106011 0.295512; visual mesh filename=meshes/left_shin_stripe.stl
- link left_thigh_clamshell: geometry collision box size=0.163304 0.067435 0.3773; visual mesh filename=meshes/left_thigh_clamshell.stl
- link left_thigh_edge: geometry collision box size=0.020824 0.018385 0.260337; visual mesh filename=meshes/left_thigh_edge.stl
- link left_thigh_ridge: geometry collision box size=0.024705 0.061015 0.25287; visual mesh filename=meshes/left_thigh_ridge.stl
- link left_thigh_shell: geometry collision box size=0.222533 0.202434 0.3773; visual mesh filename=meshes/left_thigh_shell.stl
- link left_thigh_stripe: geometry collision box size=0.040318 0.176468 0.271656; visual mesh filename=meshes/left_thigh_stripe.stl
- link right_bicep_clamshell: geometry collision box size=0.109834 0.043318 0.26691; visual mesh filename=meshes/right_bicep_clamshell.stl
- link right_bicep_front: geometry collision box size=0.017641 0.077505 0.202852; visual mesh filename=meshes/right_bicep_front.stl
- link right_bicep_sleeve: geometry collision box size=0.14967 0.138399 0.26691; visual mesh filename=meshes/right_bicep_sleeve.stl
- link right_calf_clamshell: geometry collision box size=0.135784 0.059603 0.37884; visual mesh filename=meshes/right_calf_clamshell.stl
- link right_chest_door: geometry collision box size=0.146048 0.233043 0.204085; visual mesh filename=meshes/right_chest_door.stl
- link right_forearm_crest: geometry collision box size=0.022191 0.090293 0.177828; visual mesh filename=meshes/right_forearm_crest.stl
- link right_gauntlet_clamshell: geometry collision box size=0.100056 0.043562 0.222285; visual mesh filename=meshes/right_gauntlet_clamshell.stl
- link right_gauntlet_sleeve: geometry collision box size=0.136346 0.125376 0.222285; visual mesh filename=meshes/right_gauntlet_sleeve.stl
- link right_hand: geometry collision box size=0.09 0.07 0.03; visual box size=0.09 0.07 0.03
- link right_hand_plate: geometry collision box size=0.014302 0.083899 0.08983; visual mesh filename=meshes/right_hand_plate.stl
- link right_hip_cowl: geometry collision box size=0.174356 0.174015 0.1; visual mesh filename=meshes/right_hip_cowl.stl
- link right_lat_plate: geometry collision box size=0.161485 0.101377 0.35; visual mesh filename=meshes/right_lat_plate.stl
- link right_pectoral_trim: geometry collision box size=0.142149 0.215993 0.07783; visual mesh filename=meshes/right_pectoral_trim.stl
- link right_shin_edge: geometry collision box size=0.018447 0.020281 0.2614; visual mesh filename=meshes/right_shin_edge.stl
- link right_shin_ridge: geometry collision box size=0.023159 0.051957 0.253823; visual mesh filename=meshes/right_shin_ridge.stl
- link right_shin_shell: geometry collision box size=0.185031 0.169954 0.37884; visual mesh filename=meshes/right_shin_shell.stl
- link right_shin_stripe: geometry collision box size=0.030225 0.106011 0.295512; visual mesh filename=meshes/right_shin_stripe.stl
- link right_thigh_clamshell: geometry collision box size=0.163304 0.067467 0.3773; visual mesh filename=meshes/right_thigh_clamshell.stl
- link right_thigh_edge: geometry collision box size=0.020831 0.018381 0.260337; visual mesh filename=meshes/right_thigh_edge.stl
- link right_thigh_ridge: geometry collision box size=0.024705 0.061015 0.25287; visual mesh filename=meshes/right_thigh_ridge.stl
- link right_thigh_shell: geometry collision box size=0.222533 0.202434 0.3773; visual mesh filename=meshes/right_thigh_shell.stl
- link right_thigh_stripe: geometry collision box size=0.040318 0.176468 0.271656; visual mesh filename=meshes/right_thigh_stripe.stl
Joints:
- joint back_shell_mount: origin xyz=-0.29 0 0.33772 rpy=0 0 3.141593 -> xyz=-0.335 0 0.33772 rpy=0 0 3.141593
- joint chest_centre_mount: origin xyz=0.204 0 0.37772 rpy=0 0 0 -> xyz=0.214 0 0.37772 rpy=0 0 0
- joint left_ankle_flap_hinge: origin xyz=0 0.085 0.02 rpy=0 0 1.570796 -> xyz=0 0.095 0.02 rpy=0 0 1.570796
- joint left_elbow_cap_hinge: origin xyz=-0.055 -0.05 0 rpy=0 -1.570796 0 -> xyz=-0.068 -0.05 0 rpy=0 -1.570796 0
- joint left_hand_plate_mount: origin xyz=0.035 -0.045 -0.017 rpy=0 -1.570796 0 -> xyz=0.05 -0.045 -0.017 rpy=0 -1.570796 0
- joint left_knee_cap_hinge: origin xyz=0.085 -0.045 0 rpy=0 0 0 -> xyz=0.11 -0.045 0 rpy=0 0 0
- joint left_palm_repulsor_mount: origin xyz=0.03 -0.045 -0.056 rpy=3.141593 0 0 -> xyz=0.045 -0.045 -0.056 rpy=3.141593 0 0
- joint left_thruster_cover_hinge: origin xyz=-0.145 -0.045 -0.02 rpy=0 0 3.141593 -> xyz=-0.18 -0.045 -0.02 rpy=0 0 3.141593
- joint right_ankle_flap_hinge: origin xyz=0 -0.085 0.02 rpy=0 0 -1.570796 -> xyz=0 -0.095 0.02 rpy=0 0 -1.570796
- joint right_elbow_cap_hinge: origin xyz=-0.055 0.05 0 rpy=0 -1.570796 0 -> xyz=-0.068 0.05 0 rpy=0 -1.570796 0
- joint right_hand_plate_mount: origin xyz=0.035 0.045 -0.017 rpy=0 -1.570796 0 -> xyz=0.05 0.045 -0.017 rpy=0 -1.570796 0
- joint right_knee_cap_hinge: origin xyz=0.085 0.045 0 rpy=0 0 0 -> xyz=0.11 0.045 0 rpy=0 0 0
- joint right_palm_repulsor_mount: origin xyz=0.03 0.045 -0.056 rpy=3.141593 0 0 -> xyz=0.045 0.045 -0.056 rpy=3.141593 0 0
- joint right_thruster_cover_hinge: origin xyz=-0.145 0.045 -0.02 rpy=0 0 3.141593 -> xyz=-0.18 0.045 -0.02 rpy=0 0 3.141593

File: examples/14_iron_man_mark_43/robot.urdf (robot description, URDF)
Before this commit: robot iron_man_mark_43, 268 links, 267 joints
Links:
- link ab_plate_3: geometry collision box size=0.018372 0.20326 0.043; visual mesh filename=package://iron_man_mark_43/meshes/ab_plate_3.stl
- link chest_plate: geometry collision box size=0.02 0.16 0.24; visual box size=0.02 0.16 0.24
- link left_bicep_clamshell: geometry collision box size=0.109834 0.043268 0.26691; visual mesh filename=package://iron_man_mark_43/meshes/left_bicep_clamshell.stl
- link left_bicep_front: geometry collision box size=0.017641 0.077505 0.202852; visual mesh filename=package://iron_man_mark_43/meshes/left_bicep_front.stl
- link left_bicep_sleeve: geometry collision box size=0.14967 0.138399 0.26691; visual mesh filename=package://iron_man_mark_43/meshes/left_bicep_sleeve.stl
- link left_calf_clamshell: geometry collision box size=0.135784 0.059588 0.37884; visual mesh filename=package://iron_man_mark_43/meshes/left_calf_clamshell.stl
- link left_chest_door: geometry collision box size=0.146048 0.233043 0.204085; visual mesh filename=package://iron_man_mark_43/meshes/left_chest_door.stl
- link left_forearm_crest: geometry collision box size=0.022191 0.090293 0.177828; visual mesh filename=package://iron_man_mark_43/meshes/left_forearm_crest.stl
- link left_gauntlet_clamshell: geometry collision box size=0.100056 0.043404 0.222285; visual mesh filename=package://iron_man_mark_43/meshes/left_gauntlet_clamshell.s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
- link left_gauntlet_sleeve: geometry collision box size=0.136346 0.125376 0.222285; visual mesh filename=package://iron_man_mark_43/meshes/left_gauntlet_sleeve.stl
- link left_hand: geometry collision box size=0.09 0.07 0.03; visual box size=0.09 0.07 0.03
- link left_hand_plate: geometry collision box size=0.014302 0.083899 0.08983; visual mesh filename=package://iron_man_mark_43/meshes/left_hand_plate.stl
- link left_hip_cowl: geometry collision box size=0.174356 0.174015 0.1; visual mesh filename=package://iron_man_mark_43/meshes/left_hip_cowl.stl
- link left_lat_plate: geometry collision box size=0.161485 0.101377 0.35; visual mesh filename=package://iron_man_mark_43/meshes/left_lat_plate.stl
- link left_pectoral_trim: geometry collision box size=0.142149 0.215993 0.07783; visual mesh filename=package://iron_man_mark_43/meshes/left_pectoral_trim.stl
- link left_shin_edge: geometry collision box size=0.018441 0.020286 0.2614; visual mesh filename=package://iron_man_mark_43/meshes/left_shin_edge.stl
- link left_shin_ridge: geometry collision box size=0.023159 0.051957 0.253823; visual mesh filename=package://iron_man_mark_43/meshes/left_shin_ridge.stl
- link left_shin_shell: geometry collision box size=0.185031 0.169954 0.37884; visual mesh filename=package://iron_man_mark_43/meshes/left_shin_shell.stl
- link left_shin_stripe: geometry collision box size=0.030225 0.106011 0.295512; visual mesh filename=package://iron_man_mark_43/meshes/left_shin_stripe.stl
- link left_thigh_clamshell: geometry collision box size=0.163304 0.067435 0.3773; visual mesh filename=package://iron_man_mark_43/meshes/left_thigh_clamshell.stl
- link left_thigh_edge: geometry collision box size=0.020824 0.018385 0.260337; visual mesh filename=package://iron_man_mark_43/meshes/left_thigh_edge.stl
- link left_thigh_ridge: geometry collision box size=0.024705 0.061015 0.25287; visual mesh filename=package://iron_man_mark_43/meshes/left_thigh_ridge.stl
- link left_thigh_shell: geometry collision box size=0.222533 0.202434 0.3773; visual mesh filename=package://iron_man_mark_43/meshes/left_thigh_shell.stl
- link left_thigh_stripe: geometry collision box size=0.040318 0.176468 0.271656; visual mesh filename=package://iron_man_mark_43/meshes/left_thigh_stripe.stl
- link right_bicep_clamshell: geometry collision box size=0.109834 0.043318 0.26691; visual mesh filename=package://iron_man_mark_43/meshes/right_bicep_clamshell.stl
- link right_bicep_front: geometry collision box size=0.017641 0.077505 0.202852; visual mesh filename=package://iron_man_mark_43/meshes/right_bicep_front.stl
- link right_bicep_sleeve: geometry collision box size=0.14967 0.138399 0.26691; visual mesh filename=package://iron_man_mark_43/meshes/right_bicep_sleeve.stl
- link right_calf_clamshell: geometry collision box size=0.135784 0.059603 0.37884; visual mesh filename=package://iron_man_mark_43/meshes/right_calf_clamshell.stl
- link right_chest_door: geometry collision box size=0.146048 0.233043 0.204085; visual mesh filename=package://iron_man_mark_43/meshes/right_chest_door.stl
- link right_forearm_crest: geometry collision box size=0.022191 0.090293 0.177828; visual mesh filename=package://iron_man_mark_43/meshes/right_forearm_crest.stl
- link right_gauntlet_clamshell: geometry collision box size=0.100056 0.043562 0.222285; visual mesh filename=package://iron_man_mark_43/meshes/right_gauntlet_clamshell.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
- link right_gauntlet_sleeve: geometry collision box size=0.136346 0.125376 0.222285; visual mesh filename=package://iron_man_mark_43/meshes/right_gauntlet_sleeve.stl
- link right_hand: geometry collision box size=0.09 0.07 0.03; visual box size=0.09 0.07 0.03
- link right_hand_plate: geometry collision box size=0.014302 0.083899 0.08983; visual mesh filename=package://iron_man_mark_43/meshes/right_hand_plate.stl
- link right_hip_cowl: geometry collision box size=0.174356 0.174015 0.1; visual mesh filename=package://iron_man_mark_43/meshes/right_hip_cowl.stl
- link right_lat_plate: geometry collision box size=0.161485 0.101377 0.35; visual mesh filename=package://iron_man_mark_43/meshes/right_lat_plate.stl
- link right_pectoral_trim: geometry collision box size=0.142149 0.215993 0.07783; visual mesh filename=package://iron_man_mark_43/meshes/right_pectoral_trim.stl
- link right_shin_edge: geometry collision box size=0.018447 0.020281 0.2614; visual mesh filename=package://iron_man_mark_43/meshes/right_shin_edge.stl
- link right_shin_ridge: geometry collision box size=0.023159 0.051957 0.253823; visual mesh filename=package://iron_man_mark_43/meshes/right_shin_ridge.stl
- link right_shin_shell: geometry collision box size=0.185031 0.169954 0.37884; visual mesh filename=package://iron_man_mark_43/meshes/right_shin_shell.stl
- link right_shin_stripe: geometry collision box size=0.030225 0.106011 0.295512; visual mesh filename=package://iron_man_mark_43/meshes/right_shin_stripe.stl
- link right_thigh_clamshell: geometry collision box size=0.163304 0.067467 0.3773; visual mesh filename=package://iron_man_mark_43/meshes/right_thigh_clamshell.stl
- link right_thigh_edge: geometry collision box size=0.020831 0.018381 0.260337; visual mesh filename=package://iron_man_mark_43/meshes/right_thigh_edge.stl
- link right_thigh_ridge: geometry collision box size=0.024705 0.061015 0.25287; visual mesh filename=package://iron_man_mark_43/meshes/right_thigh_ridge.stl
- link right_thigh_shell: geometry collision box size=0.222533 0.202434 0.3773; visual mesh filename=package://iron_man_mark_43/meshes/right_thigh_shell.stl
- link right_thigh_stripe: geometry collision box size=0.040318 0.176468 0.271656; visual mesh filename=package://iron_man_mark_43/meshes/right_thigh_stripe.stl
Joints:
- joint back_shell_mount: origin xyz=-0.29 0 0.33772 rpy=0 0 3.141593 -> xyz=-0.335 0 0.33772 rpy=0 0 3.141593
- joint chest_centre_mount: origin xyz=0.204 0 0.37772 rpy=0 0 0 -> xyz=0.214 0 0.37772 rpy=0 0 0
- joint left_ankle_flap_hinge: origin xyz=0 0.085 0.02 rpy=0 0 1.570796 -> xyz=0 0.095 0.02 rpy=0 0 1.570796
- joint left_elbow_cap_hinge: origin xyz=-0.055 -0.05 0 rpy=0 -1.570796 0 -> xyz=-0.068 -0.05 0 rpy=0 -1.570796 0
- joint left_hand_plate_mount: origin xyz=0.035 -0.045 -0.017 rpy=0 -1.570796 0 -> xyz=0.05 -0.045 -0.017 rpy=0 -1.570796 0
- joint left_knee_cap_hinge: origin xyz=0.085 -0.045 0 rpy=0 0 0 -> xyz=0.11 -0.045 0 rpy=0 0 0
- joint left_palm_repulsor_mount: origin xyz=0.03 -0.045 -0.056 rpy=3.141593 0 0 -> xyz=0.045 -0.045 -0.056 rpy=3.141593 0 0
- joint left_thruster_cover_hinge: origin xyz=-0.145 -0.045 -0.02 rpy=0 0 3.141593 -> xyz=-0.18 -0.045 -0.02 rpy=0 0 3.141593
- joint right_ankle_flap_hinge: origin xyz=0 -0.085 0.02 rpy=0 0 -1.570796 -> xyz=0 -0.095 0.02 rpy=0 0 -1.570796
- joint right_elbow_cap_hinge: origin xyz=-0.055 0.05 0 rpy=0 -1.570796 0 -> xyz=-0.068 0.05 0 rpy=0 -1.570796 0
- joint right_hand_plate_mount: origin xyz=0.035 0.045 -0.017 rpy=0 -1.570796 0 -> xyz=0.05 0.045 -0.017 rpy=0 -1.570796 0
- joint right_knee_cap_hinge: origin xyz=0.085 0.045 0 rpy=0 0 0 -> xyz=0.11 0.045 0 rpy=0 0 0
- joint right_palm_repulsor_mount: origin xyz=0.03 0.045 -0.056 rpy=3.141593 0 0 -> xyz=0.045 0.045 -0.056 rpy=3.141593 0 0
- joint right_thruster_cover_hinge: origin xyz=-0.145 0.045 -0.02 rpy=0 0 3.141593 -> xyz=-0.18 0.045 -0.02 rpy=0 0 3.141593

Commit message: Fix Mark 43 early chest-opening interference and strengthen motion checks

File: examples/14_iron_man_mark_43/robot.sim.urdf (robot description, URDF)
Before this commit: robot iron_man_mark_43, 268 links, 267 joints
Links:
- link left_chest_door: geometry collision box size=0.143405 0.202353 0.204085; visual mesh filename=meshes/left_chest_door.stl
- link left_pectoral_trim: geometry collision box size=0.139962 0.185718 0.0779; visual mesh filename=meshes/left_pectoral_trim.stl
- link right_chest_door: geometry collision box size=0.143405 0.202353 0.204085; visual mesh filename=meshes/right_chest_door.stl
- link right_pectoral_trim: geometry collision box size=0.139962 0.185718 0.0779; visual mesh filename=meshes/right_pectoral_trim.stl

File: examples/14_iron_man_mark_43/robot.urdf (robot description, URDF)
Before this commit: robot iron_man_mark_43, 268 links, 267 joints
Links:
- link left_chest_door: geometry collision box size=0.143405 0.202353 0.204085; visual mesh filename=package://iron_man_mark_43/meshes/left_chest_door.stl
- link left_pectoral_trim: geometry collision box size=0.139962 0.185718 0.0779; visual mesh filename=package://iron_man_mark_43/meshes/left_pectoral_trim.stl
- link right_chest_door: geometry collision box size=0.143405 0.202353 0.204085; visual mesh filename=package://iron_man_mark_43/meshes/right_chest_door.stl
- link right_pectoral_trim: geometry collision box size=0.139962 0.185718 0.0779; visual mesh filename=package://iron_man_mark_43/meshes/right_pectoral_trim.stl

Commit message: Correct Mark 43 neck and opening directions; audit every joint

File: examples/14_iron_man_mark_43/robot.sim.urdf (robot description, URDF)
Before this commit: robot iron_man_mark_43, 268 links, 267 joints
Links:
- link neck_ring: mass 0.3 -> 0.156; geometry collision box size=0.16 0.16 0.013; visual mesh filename=meshes/neck_ring.stl
Joints:
- joint collar_plate_mount: origin xyz=0.135 0 0.539 rpy=0 0 0 -> xyz=0.135 0 0.531 rpy=0 0 0
- joint helmet_neck_collar_mount: origin xyz=0.02 0 0.71075 rpy=0 0 0 -> xyz=0 0 0.105 rpy=0 0 0; parent spine_frame -> neck_yaw_carrier
- joint left_bicep_clamshell_hinge: limit lower=-1.4 upper=0 effort=3 velocity=3 -> lower=0 upper=1.4 effort=3 velocity=3
- joint left_calf_clamshell_hinge: limit lower=-1.4 upper=0 effort=3 velocity=3 -> lower=0 upper=1.4 effort=3 velocity=3
- joint left_gauntlet_clamshell_hinge: limit lower=-1.4 upper=0 effort=3 velocity=3 -> lower=0 upper=1.4 effort=3 velocity=3
- joint left_thigh_clamshell_hinge: limit lower=-1.4 upper=0 effort=3 velocity=3 -> lower=0 upper=1.4 effort=3 velocity=3
- joint neck_ring_mount: origin xyz=0.02 0 0.556 rpy=0 0 0 -> xyz=0.02 0 0.55 rpy=0 0 0
- joint right_bicep_clamshell_hinge: limit lower=0 upper=1.4 effort=3 velocity=3 -> lower=-1.4 upper=0 effort=3 velocity=3
- joint right_calf_clamshell_hinge: limit lower=0 upper=1.4 effort=3 velocity=3 -> lower=-1.4 upper=0 effort=3 velocity=3
- joint right_gauntlet_clamshell_hinge: limit lower=0 upper=1.4 effort=3 velocity=3 -> lower=-1.4 upper=0 effort=3 velocity=3
- joint right_thigh_clamshell_hinge: limit lower=0 upper=1.4 effort=3 velocity=3 -> lower=-1.4 upper=0 effort=3 velocity=3

File: examples/14_iron_man_mark_43/robot.urdf (robot description, URDF)
Before this commit: robot iron_man_mark_43, 268 links, 267 joints
Links:
- link neck_ring: mass 0.3 -> 0.156; geometry collision box size=0.16 0.16 0.013; visual mesh filename=package://iron_man_mark_43/meshes/neck_ring.stl
Joints:
- joint collar_plate_mount: origin xyz=0.135 0 0.539 rpy=0 0 0 -> xyz=0.135 0 0.531 rpy=0 0 0
- joint helmet_neck_collar_mount: origin xyz=0.02 0 0.71075 rpy=0 0 0 -> xyz=0 0 0.105 rpy=0 0 0; parent spine_frame -> neck_yaw_carrier
- joint left_bicep_clamshell_hinge: limit lower=-1.4 upper=0 effort=3 velocity=3 -> lower=0 upper=1.4 effort=3 velocity=3
- joint left_calf_clamshell_hinge: limit lower=-1.4 upper=0 effort=3 velocity=3 -> lower=0 upper=1.4 effort=3 velocity=3
- joint left_gauntlet_clamshell_hinge: limit lower=-1.4 upper=0 effort=3 velocity=3 -> lower=0 upper=1.4 effort=3 velocity=3
- joint left_thigh_clamshell_hinge: limit lower=-1.4 upper=0 effort=3 velocity=3 -> lower=0 upper=1.4 effort=3 velocity=3
- joint neck_ring_mount: origin xyz=0.02 0 0.556 rpy=0 0 0 -> xyz=0.02 0 0.55 rpy=0 0 0
- joint right_bicep_clamshell_hinge: limit lower=0 upper=1.4 effort=3 velocity=3 -> lower=-1.4 upper=0 effort=3 velocity=3
- joint right_calf_clamshell_hinge: limit lower=0 upper=1.4 effort=3 velocity=3 -> lower=-1.4 upper=0 effort=3 velocity=3
- joint right_gauntlet_clamshell_hinge: limit lower=0 upper=1.4 effort=3 velocity=3 -> lower=-1.4 upper=0 effort=3 velocity=3
- joint right_thigh_clamshell_hinge: limit lower=0 upper=1.4 effort=3 velocity=3 -> lower=-1.4 upper=0 effort=3 velocity=3
