Commit message: feat: articulated Iron Man Mark suit -- 45 hinged armour plates, donning sequence, proportioned wearer
The suit is now a Mark suit in the mechanical sense: a wearable exoskeleton under
armour that opens to let the wearer in and locks closed, every moving part a real
hinged, actuated link, simulated with a properly proportioned person inside.

- templates/marksuit.ts: ironManMarkSuit -- 45 servo-driven armour hinges on top
  of the 17-joint frame (faceplate, chest halves, back doors, air-brake flaps,
  folding ab segments, codpiece, pauldrons, bicep/forearm clamshells, gauntlet
  hatches, fingers + thumbs, hip flaps, thigh/calf clamshells, knee caps, shin
  guards, thruster covers, ankle flaps); 111 links, 62 actuators, 76.6 kg.
  Routing: iron man / mark / armour -> Mark suit; bare exoskeleton wording ->
  exosuit; battle mech -> humanoid. anthropometrics() exported.
- python: renderer motions don/doff/open drive *_hinge servos in anatomical
  order (boots -> legs -> torso -> arms -> faceplate); --orbit/--azimuth/--zoom/
  --width/--height/--fps. Wearer mannequin rebuilt as a proportioned adult
  (neck, clavicles, chest + abdomen, tapered limbs, hands, feet).
- results (suit + 75 kg wearer, 151 kg): battery 5/5, wearer support 5 mm vs
  1.39 m collapse, donning closes 45/45 plates within 0.001 rad upright; a
  1 m/s shove leans it to 0.46 (documented). BOM ~$44.7k research tier.
- fix: tiny parts produced degenerate inertia tensors through 6-decimal URDF
  formatting (MuJoCo rejected them); num() now keeps 6 significant figures for
  small values and finalize floors principal moments.
- README rewritten around the donning sequence with five MuJoCo GIFs; all 17
  examples regenerated (17/17 PyBullet, all MuJoCo reports refreshed); 70 tests

File: examples/11_spider_scout/robot.urdf (robot description, URDF)
Before this commit: robot hexapod, 20 links, 19 joints
Joints:
- joint mid_right_coxa_joint: origin xyz=-0.15 0 0.18 rpy=0 0 3.141593 -> xyz=-0.15 1.83697e-17 0.18 rpy=0 0 3.141593

File: examples/15_wall_e/robot.urdf (robot description, URDF)
Before this commit: robot wall_e, 24 links, 23 joints
Links:
- removed link camera_3_link
Joints:
- removed joint camera_3_joint

Commit message: Harden the parser against adversarial prompts and mount sensors on the body surface
An adversarial sweep (~330 prompts, ~200 edits) found 28 misreadings; all fixed with tests.

Parser: doesn't/neither-nor/postfix/"instead of" negation and "no sensors except X";
negating a sensor no longer hides the robot type; payload only when a payload word is
adjacent ("picks up 2 kg boxes"), robot mass reported separately; size words must describe
the robot, not objects or names; names and quoted text are masked from feature parsing;
"robot with 4 legs/wheels"; suction on mobile manipulators and SCARA grippers; arms on
legged bases, unmodelled sensors and fixed-size templates are reported; "1,000 mm",
"one metre", 3' reach; positions are not reach; "5 grand", "2000$"; colour forms
("colour: red", "(blue)", "golden"); sensor counts and per-sensor locations.

Edits: relative DOF ("add two joints"); sensors before grippers ("camera on the gripper");
shared predicates and exclusions ("forearm and upper arm 10% longer", "but not the upper
arm", "keep the camera", "everything except"); both humanoid hands swap grippers; legs,
character liveries and suit limbs refuse clearly; suits refit to a new wearer; renames keep
the whole name; polite prefixes, "longer.add" and budgets alongside other edits.

Sensors are placed on the outer surface of the assembled body (lidars on top, cameras at
the front or wrist, IMUs inside) instead of 5 cm above the link origin, where they were
buried in the chassis. Examples 11 and 12 are regenerated: same MuJoCo results (6/6, 5/6),
zero initial penetrations, ROS 2 Jazzy colcon rebuild, training, mobile-motion and browser
records refreshed with MuJoCo 3.13.0; verify_example_artifacts passes.

CLI help no longer advertises removed cloud API keys.

File: examples/11_spider_scout/robot.urdf (robot description, URDF)
Before this commit: robot hexapod, 35 links, 34 joints
Joints:
- joint lidar_1_joint: origin xyz=0 0 0.05 rpy=0 0 0 -> xyz=0 0 0.165 rpy=0 0 0

File: examples/12_mars_rover/robot.urdf (robot description, URDF)
Before this commit: robot rover_arm, 44 links, 43 joints
Joints:
- joint camera_1_joint: origin xyz=0 0 0.05 rpy=0 0 0 -> xyz=-0.18 0 0.195 rpy=0 0 0
- joint depth_1_joint: origin xyz=0 0 0.05 rpy=0 0 0 -> xyz=0.18 0 0.195 rpy=0 0 0
