Commit message: feat: MoveIt 2 + Gazebo export, native STL + printability, share links, verified training
Hardening pass toward a complete, self-hostable free service.

- cad: native STL triangulation (box/cylinder/sphere/capsule) per link + assembly,
  no OpenSCAD required; printability report (build volume, thin features)
- ros2-export: MoveIt 2 config (SRDF chain + gripper group, kinematics, controllers,
  OMPL, move_group launch) and Gazebo (gz-sim world + ros_gz spawn launch)
- api/web: persistent robot store (data/robots.json), shareable /r/<id> links that
  restore the robot, Share button; Dockerfile + .dockerignore for one-command hosting
- templates: humanoid rebuilt with coherent frames and 3-DOF legs (stands on the
  ground, shoulders at torso top, classifies as locomotion)
- web: fix HiDPI canvas overflow (setSize must update CSS size) -- layout was broken
  on Retina/DPR-2 displays
- cli: fix argument parsing bug where a missing -o dropped the subcommand, making
  `validate` silently generate; default output now ./out/<name>/ (gitignored);
  CLI regression tests
- training-export: trainer tolerates a missing tensorboard; suite executed end to
  end in PyBullet (env for every class, demos -> PPO/SAC -> BC -> evaluate)
- scripts/physics_check.py: every example loads and simulates in PyBullet (13/13)
- strict TypeScript typecheck clean (tsconfig, npm run typecheck); 55 tests
- README/ARCHITECTURE: screenshots re-captured at HiDPI, new sections, roadmap

File: examples/08_humanoid/robot.urdf (robot description, URDF)
Before this commit: robot humanoid_robot, 22 links, 21 joints
Links:
- added link left_foot, mass 0.2304; collision box size=0.16 0.08 0.04; visual box size=0.16 0.08 0.04
- added link left_shin, mass 0.452389; collision cylinder length=0.2 radius=0.04; visual cylinder length=0.2 radius=0.04
- added link left_thigh, mass 0.572555; collision cylinder length=0.2 radius=0.045; visual cylinder length=0.2 radius=0.045
- added link right_foot, mass 0.2304; collision box size=0.16 0.08 0.04; visual box size=0.16 0.08 0.04
- added link right_shin, mass 0.452389; collision cylinder length=0.2 radius=0.04; visual cylinder length=0.2 radius=0.04
- added link right_thigh, mass 0.572555; collision cylinder length=0.2 radius=0.045; visual cylinder length=0.2 radius=0.045
Joints:
- removed joint left_joint_1
- removed joint left_joint_2
- removed joint left_joint_3
- removed joint left_joint_4
- removed joint left_joint_5
- removed joint left_joint_6
- removed joint left_joint_7
- removed joint right_joint_1
- removed joint right_joint_2
- removed joint right_joint_3
- removed joint right_joint_4
- removed joint right_joint_5
- removed joint right_joint_6
- removed joint right_joint_7
- added joint left_ankle_joint: type revolute, parent left_shin, child left_foot, origin xyz=0 0 -0.2 rpy=0 0 0, axis 0 1 0, limit lower=-0.8 upper=0.8 effort=50 velocity=2
- added joint left_arm_joint_1: type revolute, parent torso, child left_shoulder, origin xyz=0 0.175 0.77 rpy=0 0 0, axis 0 1 0, limit lower=-2.6 upper=2.6 effort=50 velocity=2
- added joint left_arm_joint_2: type revolute, parent left_shoulder, child left_upper_arm, origin xyz=0 0 -0.06 rpy=0 0 0, axis 1 0 0, limit lower=-2.6 upper=2.6 effort=50 velocity=2
- added joint left_arm_joint_3: type revolute, parent left_upper_arm, child left_elbow, origin xyz=0 0 -0.22 rpy=0 0 0, axis 0 1 0, limit lower=-2.6 upper=2.6 effort=50 velocity=2
- added joint left_arm_joint_4: type revolute, parent left_elbow, child left_forearm, origin xyz=0 0 -0.06 rpy=0 0 0, axis 1 0 0, limit lower=-2.6 upper=2.6 effort=50 velocity=2
- added joint left_arm_joint_5: type revolute, parent left_forearm, child left_wrist_1, origin xyz=0 0 -0.22 rpy=0 0 0, axis 0 1 0, limit lower=-2.6 upper=2.6 effort=50 velocity=2
- added joint left_arm_joint_6: type revolute, parent left_wrist_1, child left_wrist_2, origin xyz=0 0 -0.06 rpy=0 0 0, axis 1 0 0, limit lower=-2.6 upper=2.6 effort=50 velocity=2
- added joint left_arm_joint_7: type revolute, parent left_wrist_2, child left_wrist_3, origin xyz=0 0 -0.06 rpy=0 0 0, axis 0 1 0, limit lower=-2.6 upper=2.6 effort=50 velocity=2
- added joint left_hip_joint: type revolute, parent torso, child left_thigh, origin xyz=0 0.07 0.44 rpy=0 0 0, axis 0 1 0, limit lower=-1.6 upper=1.6 effort=50 velocity=2
- added joint left_knee_joint: type revolute, parent left_thigh, child left_shin, origin xyz=0 0 -0.2 rpy=0 0 0, axis 0 1 0, limit lower=0 upper=2.4 effort=50 velocity=2
- added joint right_ankle_joint: type revolute, parent right_shin, child right_foot, origin xyz=0 0 -0.2 rpy=0 0 0, axis 0 1 0, limit lower=-0.8 upper=0.8 effort=50 velocity=2
- added joint right_arm_joint_1: type revolute, parent torso, child right_shoulder, origin xyz=0 -0.175 0.77 rpy=0 0 0, axis 0 1 0, limit lower=-2.6 upper=2.6 effort=50 velocity=2
- added joint right_arm_joint_2: type revolute, parent right_shoulder, child right_upper_arm, origin xyz=0 0 -0.06 rpy=0 0 0, axis 1 0 0, limit lower=-2.6 upper=2.6 effort=50 velocity=2
- added joint right_arm_joint_3: type revolute, parent right_upper_arm, child right_elbow, origin xyz=0 0 -0.22 rpy=0 0 0, axis 0 1 0, limit lower=-2.6 upper=2.6 effort=50 velocity=2
- added joint right_arm_joint_4: type revolute, parent right_elbow, child right_forearm, origin xyz=0 0 -0.06 rpy=0 0 0, axis 1 0 0, limit lower=-2.6 upper=2.6 effort=50 velocity=2
- added joint right_arm_joint_5: type revolute, parent right_forearm, child right_wrist_1, origin xyz=0 0 -0.22 rpy=0 0 0, axis 0 1 0, limit lower=-2.6 upper=2.6 effort=50 velocity=2
- added joint right_arm_joint_6: type revolute, parent right_wrist_1, child right_wrist_2, origin xyz=0 0 -0.06 rpy=0 0 0, axis 1 0 0, limit lower=-2.6 upper=2.6 effort=50 velocity=2
- added joint right_arm_joint_7: type revolute, parent right_wrist_2, child right_wrist_3, origin xyz=0 0 -0.06 rpy=0 0 0, axis 0 1 0, limit lower=-2.6 upper=2.6 effort=50 velocity=2
- added joint right_hip_joint: type revolute, parent torso, child right_thigh, origin xyz=0 -0.07 0.44 rpy=0 0 0, axis 0 1 0, limit lower=-1.6 upper=1.6 effort=50 velocity=2
- added joint right_knee_joint: type revolute, parent right_thigh, child right_shin, origin xyz=0 0 -0.2 rpy=0 0 0, axis 0 1 0, limit lower=0 upper=2.4 effort=50 velocity=2
- joint neck_joint: origin xyz=0 0 1.05 rpy=0 0 0 -> xyz=0 0 0.89 rpy=0 0 0

File: examples/13_battle_mech/robot.urdf (robot description, URDF)
Before this commit: robot humanoid_robot, 24 links, 23 joints
Links:
- added link left_foot, mass 0.2304; collision box size=0.16 0.08 0.04; visual box size=0.16 0.08 0.04
- added link left_shin, mass 0.452389; collision cylinder length=0.2 radius=0.04; visual cylinder length=0.2 radius=0.04
- added link left_thigh, mass 0.572555; collision cylinder length=0.2 radius=0.045; visual cylinder length=0.2 radius=0.045
- added link right_foot, mass 0.2304; collision box size=0.16 0.08 0.04; visual box size=0.16 0.08 0.04
- added link right_shin, mass 0.452389; collision cylinder length=0.2 radius=0.04; visual cylinder length=0.2 radius=0.04
- added link right_thigh, mass 0.572555; collision cylinder length=0.2 radius=0.045; visual cylinder length=0.2 radius=0.045
Joints:
- removed joint left_joint_1
- removed joint left_joint_2
- removed joint left_joint_3
- removed joint left_joint_4
- removed joint left_joint_5
- removed joint left_joint_6
- removed joint left_joint_7
- removed joint right_joint_1
- removed joint right_joint_2
- removed joint right_joint_3
- removed joint right_joint_4
- removed joint right_joint_5
- removed joint right_joint_6
- removed joint right_joint_7
- added joint left_ankle_joint: type revolute, parent left_shin, child left_foot, origin xyz=0 0 -0.2 rpy=0 0 0, axis 0 1 0, limit lower=-0.8 upper=0.8 effort=50 velocity=2
- added joint left_arm_joint_1: type revolute, parent torso, child left_shoulder, origin xyz=0 0.175 0.77 rpy=0 0 0, axis 0 1 0, limit lower=-2.6 upper=2.6 effort=50 velocity=2
- added joint left_arm_joint_2: type revolute, parent left_shoulder, child left_upper_arm, origin xyz=0 0 -0.06 rpy=0 0 0, axis 1 0 0, limit lower=-2.6 upper=2.6 effort=50 velocity=2
- added joint left_arm_joint_3: type revolute, parent left_upper_arm, child left_elbow, origin xyz=0 0 -0.22 rpy=0 0 0, axis 0 1 0, limit lower=-2.6 upper=2.6 effort=50 velocity=2
- added joint left_arm_joint_4: type revolute, parent left_elbow, child left_forearm, origin xyz=0 0 -0.06 rpy=0 0 0, axis 1 0 0, limit lower=-2.6 upper=2.6 effort=50 velocity=2
- added joint left_arm_joint_5: type revolute, parent left_forearm, child left_wrist_1, origin xyz=0 0 -0.22 rpy=0 0 0, axis 0 1 0, limit lower=-2.6 upper=2.6 effort=50 velocity=2
- added joint left_arm_joint_6: type revolute, parent left_wrist_1, child left_wrist_2, origin xyz=0 0 -0.06 rpy=0 0 0, axis 1 0 0, limit lower=-2.6 upper=2.6 effort=50 velocity=2
- added joint left_arm_joint_7: type revolute, parent left_wrist_2, child left_wrist_3, origin xyz=0 0 -0.06 rpy=0 0 0, axis 0 1 0, limit lower=-2.6 upper=2.6 effort=50 velocity=2
- added joint left_hip_joint: type revolute, parent torso, child left_thigh, origin xyz=0 0.07 0.44 rpy=0 0 0, axis 0 1 0, limit lower=-1.6 upper=1.6 effort=50 velocity=2
- added joint left_knee_joint: type revolute, parent left_thigh, child left_shin, origin xyz=0 0 -0.2 rpy=0 0 0, axis 0 1 0, limit lower=0 upper=2.4 effort=50 velocity=2
- added joint right_ankle_joint: type revolute, parent right_shin, child right_foot, origin xyz=0 0 -0.2 rpy=0 0 0, axis 0 1 0, limit lower=-0.8 upper=0.8 effort=50 velocity=2
- added joint right_arm_joint_1: type revolute, parent torso, child right_shoulder, origin xyz=0 -0.175 0.77 rpy=0 0 0, axis 0 1 0, limit lower=-2.6 upper=2.6 effort=50 velocity=2
- added joint right_arm_joint_2: type revolute, parent right_shoulder, child right_upper_arm, origin xyz=0 0 -0.06 rpy=0 0 0, axis 1 0 0, limit lower=-2.6 upper=2.6 effort=50 velocity=2
- added joint right_arm_joint_3: type revolute, parent right_upper_arm, child right_elbow, origin xyz=0 0 -0.22 rpy=0 0 0, axis 0 1 0, limit lower=-2.6 upper=2.6 effort=50 velocity=2
- added joint right_arm_joint_4: type revolute, parent right_elbow, child right_forearm, origin xyz=0 0 -0.06 rpy=0 0 0, axis 1 0 0, limit lower=-2.6 upper=2.6 effort=50 velocity=2
- added joint right_arm_joint_5: type revolute, parent right_forearm, child right_wrist_1, origin xyz=0 0 -0.22 rpy=0 0 0, axis 0 1 0, limit lower=-2.6 upper=2.6 effort=50 velocity=2
- added joint right_arm_joint_6: type revolute, parent right_wrist_1, child right_wrist_2, origin xyz=0 0 -0.06 rpy=0 0 0, axis 1 0 0, limit lower=-2.6 upper=2.6 effort=50 velocity=2
- added joint right_arm_joint_7: type revolute, parent right_wrist_2, child right_wrist_3, origin xyz=0 0 -0.06 rpy=0 0 0, axis 0 1 0, limit lower=-2.6 upper=2.6 effort=50 velocity=2
- added joint right_hip_joint: type revolute, parent torso, child right_thigh, origin xyz=0 -0.07 0.44 rpy=0 0 0, axis 0 1 0, limit lower=-1.6 upper=1.6 effort=50 velocity=2
- added joint right_knee_joint: type revolute, parent right_thigh, child right_shin, origin xyz=0 0 -0.2 rpy=0 0 0, axis 0 1 0, limit lower=0 upper=2.4 effort=50 velocity=2
- joint neck_joint: origin xyz=0 0 1.05 rpy=0 0 0 -> xyz=0 0 0.89 rpy=0 0 0

Commit message: Regenerate 08_humanoid and refresh the evidence that depends on it
08_humanoid rebuilt from its prompt with the shortened arms: URDF, spec,
CAD/ROS/training archives, BOM, simulation report (6/7, only the 1 m/s
shove fails; standing_balance passes), GIF, MoveIt mock left-arm run and
ROS 2 Jazzy colcon build. Coordinated arm-motion reports and GIFs for
01-04 re-run because the controller and servo damping changed. Web,
training and runtime records updated for the new hashes. Other examples'
simulation reports are unchanged and were recorded with the previous
test battery.

File: examples/08_humanoid/robot.urdf (robot description, URDF)
Before this commit: robot humanoid_robot, 47 links, 46 joints
Links:
- link left_forearm: mass 0.380997 -> 0.311725; geometry collision cylinder length=0.18 radius=0.035; visual cylinder length=0.18 radius=0.035
- link left_upper_arm: mass 0.380997 -> 0.311725; geometry collision cylinder length=0.18 radius=0.035; visual cylinder length=0.18 radius=0.035
- link right_forearm: mass 0.380997 -> 0.311725; geometry collision cylinder length=0.18 radius=0.035; visual cylinder length=0.18 radius=0.035
- link right_upper_arm: mass 0.380997 -> 0.311725; geometry collision cylinder length=0.18 radius=0.035; visual cylinder length=0.18 radius=0.035
Joints:
- joint left_arm_joint_3: origin xyz=0 0 -0.22 rpy=0 0 0 -> xyz=0 0 -0.18 rpy=0 0 0
- joint left_arm_joint_5: origin xyz=0 0 -0.22 rpy=0 0 0 -> xyz=0 0 -0.18 rpy=0 0 0
- joint right_arm_joint_3: origin xyz=0 0 -0.22 rpy=0 0 0 -> xyz=0 0 -0.18 rpy=0 0 0
- joint right_arm_joint_5: origin xyz=0 0 -0.22 rpy=0 0 0 -> xyz=0 0 -0.18 rpy=0 0 0
