Commit message: New example pipeline: build_examples.ts (all deliverables from the prompt) and simulate_examples.py (task tests filmed into the GIF, README results, gallery); mesh collisions for designed robots

File: examples/02_arm_6dof/robot.urdf (robot description, URDF)
Before this commit: robot arm_6dof, 28 links, 27 joints
Links:
- removed link base_link_front_panel
- removed link base_link_left_panel
- removed link base_link_rear_panel
- removed link base_link_right_panel
- removed link base_link_service_lid
- removed link base_link_standoff_fl
- removed link base_link_standoff_fr
- removed link base_link_standoff_rl
- removed link base_link_standoff_rr
- removed link forearm_joint_hub
- removed link gripper_base
- removed link left_finger
- removed link left_finger_pad
- removed link right_finger
- removed link right_finger_pad
- removed link shoulder
- removed link shoulder_joint_hub
- removed link shoulder_mount
- removed link upper_arm_joint_hub
- removed link wrist_1
- removed link wrist_1_joint_hub
- removed link wrist_2
- removed link wrist_2_joint_hub
- removed link wrist_3
- removed link wrist_3_joint_hub
- added link base_yaw_actuator, mass 0.055; collision mesh filename=package://arm_6dof/meshes/feetech_sts3215_c047.stl; visual mesh filename=package://arm_6dof/meshes/feetech_sts3215_c047.stl
- added link elbow_pitch_actuator, mass 0.055; collision mesh filename=package://arm_6dof/meshes/feetech_sts3215_c047.stl; visual mesh filename=package://arm_6dof/meshes/feetech_sts3215_c047.stl
- added link forearm_roll_actuator, mass 0.055; collision mesh filename=package://arm_6dof/meshes/feetech_sts3215_c047.stl; visual mesh filename=package://arm_6dof/meshes/feetech_sts3215_c047.stl
- added link forearm_rotator, mass 0.016231; collision mesh filename=package://arm_6dof/meshes/forearm_rotator.stl; visual mesh filename=package://arm_6dof/meshes/forearm_rotator.stl
- added link gripper_actuator, mass 0.055; collision mesh filename=package://arm_6dof/meshes/feetech_sts3215_c047.stl; visual mesh filename=package://arm_6dof/meshes/feetech_sts3215_c047.stl
- added link gripper_jaw, mass 0.005178; collision mesh filename=package://arm_6dof/meshes/gripper_jaw.stl; visual mesh filename=package://arm_6dof/meshes/gripper_jaw.stl
- added link shoulder_pitch_actuator, mass 0.0745; collision mesh filename=package://arm_6dof/meshes/feetech_sts3250.stl; visual mesh filename=package://arm_6dof/meshes/feetech_sts3250.stl
- added link turret, mass 0.016231; collision mesh filename=package://arm_6dof/meshes/turret.stl; visual mesh filename=package://arm_6dof/meshes/turret.stl
- added link wrist, mass 0.03006; collision mesh filename=package://arm_6dof/meshes/wrist.stl; visual mesh filename=package://arm_6dof/meshes/wrist.stl
- added link wrist_pitch_actuator, mass 0.055; collision mesh filename=package://arm_6dof/meshes/feetech_sts3215_c047.stl; visual mesh filename=package://arm_6dof/meshes/feetech_sts3215_c047.stl
- added link wrist_roll_actuator, mass 0.055; collision mesh filename=package://arm_6dof/meshes/feetech_sts3215_c047.stl; visual mesh filename=package://arm_6dof/meshes/feetech_sts3215_c047.stl
- added link wrist_rotator, mass 0.024232; collision mesh filename=package://arm_6dof/meshes/wrist_rotator.stl; visual mesh filename=package://arm_6dof/meshes/wrist_rotator.stl
- link base_link: mass 0.167671 -> 0.081359; geometry collision mesh filename=package://arm_6dof/meshes/base_link.stl; visual mesh filename=package://arm_6dof/meshes/base_link.stl
- link forearm: mass 0.21879 -> 0.033199; geometry collision mesh filename=package://arm_6dof/meshes/forearm.stl; visual mesh filename=package://arm_6dof/meshes/forearm.stl
- link upper_arm: mass 0.21879 -> 0.024969; geometry collision mesh filename=package://arm_6dof/meshes/upper_arm.stl; visual mesh filename=package://arm_6dof/meshes/upper_arm.stl
Joints:
- removed joint base_link_front_panel_mount
- removed joint base_link_left_panel_mount
- removed joint base_link_rear_panel_mount
- removed joint base_link_right_panel_mount
- removed joint base_link_service_lid_mount
- removed joint base_link_standoff_fl_mount
- removed joint base_link_standoff_fr_mount
- removed joint base_link_standoff_rl_mount
- removed joint base_link_standoff_rr_mount
- removed joint forearm_joint_hub_mount
- removed joint gripper_base_joint
- removed joint joint_1
- removed joint joint_2
- removed joint joint_3
- removed joint joint_4
- removed joint joint_5
- removed joint joint_6
- removed joint left_finger_joint
- removed joint left_finger_pad_mount
- removed joint right_finger_joint
- removed joint right_finger_pad_mount
- removed joint shoulder_joint_hub_mount
- removed joint shoulder_mount_fixed
- removed joint upper_arm_joint_hub_mount
- removed joint wrist_1_joint_hub_mount
- removed joint wrist_2_joint_hub_mount
- removed joint wrist_3_joint_hub_mount
- added joint base_yaw: type revolute, parent base_link, child turret, origin xyz=0 0 0.0481 rpy=0 0 0, axis 0 0 1, limit lower=-2.97 upper=2.97 effort=2.942 velocity=4.48
- added joint base_yaw_actuator_mount: type fixed, parent base_link, child base_yaw_actuator, origin xyz=0 0 0.0481 rpy=0 0 0
- added joint elbow_pitch: type revolute, parent upper_arm, child forearm, origin xyz=0.108181 0 -0.0381 rpy=3.141593 0 0, axis 0 0 1, limit lower=-2.3 upper=2.3 effort=2.942 velocity=3.4
- added joint elbow_pitch_actuator_mount: type fixed, parent upper_arm, child elbow_pitch_actuator, origin xyz=0.108181 0 -0.0381 rpy=3.141593 0 0
- added joint forearm_roll: type revolute, parent forearm, child forearm_rotator, origin xyz=0.108181 0 -0.01905 rpy=-1.570796 0 -1.570796, axis 0 0 1, limit lower=-2.97 upper=2.97 effort=2.942 velocity=4.48
- added joint forearm_roll_actuator_mount: type fixed, parent forearm, child forearm_roll_actuator, origin xyz=0.108181 0 -0.01905 rpy=-1.570796 0 -1.570796
- added joint gripper: type revolute, parent wrist_rotator, child gripper_jaw, origin xyz=0.01905 0 0.0442 rpy=0 -1.570796 -3.141593, axis 0 0 1, limit lower=-0.35 upper=0.464 effort=2.942 velocity=4.712
- added joint gripper_actuator_mount: type fixed, parent wrist_rotator, child gripper_actuator, origin xyz=0.01905 0 0.0442 rpy=0 -1.570796 -3.141593
- added joint shoulder_pitch: type revolute, parent turret, child upper_arm, origin xyz=0 0.01905 0.0442 rpy=0 -1.570796 -1.570796, axis 0 0 1, limit lower=-1.75 upper=1.75 effort=4.9033 velocity=5.02
- added joint shoulder_pitch_actuator_mount: type fixed, parent turret, child shoulder_pitch_actuator, origin xyz=0 0.01905 0.0442 rpy=0 -1.570796 -1.570796
- added joint wrist_pitch: type revolute, parent forearm_rotator, child wrist, origin xyz=0 0.01905 0.0442 rpy=0 -1.570796 -1.570796, axis 0 0 1, limit lower=-2.3 upper=2.3 effort=2.942 velocity=4.48
- added joint wrist_pitch_actuator_mount: type fixed, parent forearm_rotator, child wrist_pitch_actuator, origin xyz=0 0.01905 0.0442 rpy=0 -1.570796 -1.570796
- added joint wrist_roll: type revolute, parent wrist, child wrist_rotator, origin xyz=0.08442 0 -0.01905 rpy=1.570796 0 1.570796, axis 0 0 1, limit lower=-2.97 upper=2.97 effort=2.942 velocity=4.48
- added joint wrist_roll_actuator_mount: type fixed, parent wrist, child wrist_roll_actuator, origin xyz=0.08442 0 -0.01905 rpy=1.570796 0 1.570796
